File: mcu.kicad_sch (KiCad schematic)
At the start: 1 part, among them U1 PIC32CK1025GC01100-I/4SB

Commit message: did stuff
Parts:
- added TP1, TP10, TP11, TP12, TP13, TP14, TP15, TP16, TP17, TP18, TP19, TP2, TP20, TP21, TP22, TP23, TP24, TP25, TP26, TP27, TP28, TP29, TP3, TP30, TP31, TP32, TP33, TP34, TP35, TP36, TP37, TP38, TP39, TP4, TP40, TP41, TP42, TP5, TP6, TP7, TP8, TP9: TestPoint, symbol Connector:TestPoint
- U1: footprint TQFP100_4SB_6p3EP_MCH -> PIC32CK1025GC01100-I-4SB:TQFP100_4SB_6p3EP_MCH
Connections:
- net +3.3V: now reaches U1.20 (VDDIO)
- net +3.3V: now also U1.33 (VDDA), U1.34 (VDDIO), U1.42 (VDDIO), U1.44 (VDDREG), U1.56 (VDDIO), U1.62 (VDDREG), U1.69 (VDDIO), U1.7 (VDDIO), U1.79 (VCCAP3), U1.83 (VDDREG), U1.85 (VDDIO), U1.96 (VDDIO)
- net SWD.SWCLK: now reaches U1.1 (PA00)
- net SWD.SWCLK: now also U1.10 (PA15), U1.11 (PA16), U1.12 (PA17), U1.14 (PA05), U1.16 (PA07), U1.17 (PA08), U1.18 (PA18), U1.2 (PA01), U1.22 (PA09), U1.23 (PA10), U1.24 (PA11), U1.25 (PA12), U1.4 (PA03), U1.51 (PC00), U1.52 (PC01), U1.54 (PC03), U1.58 (PC14), U1.59 (PC05), U1.61 (PC07), U1.63 (PC09), U1.64 (PC15), U1.65 (PC16), U1.66 (PC17), U1.67 (PC18), U1.68 (PC10), U1.71 (PC11), U1.72 (PC12), U1.73 (PC13), U1.74 (PC19), U1.8 (PA13), U1.9 (PA14), TP1.1, TP10.1, TP11.1, TP12.1, TP13.1, TP14.1, TP15.1, TP16.1, TP17.1, TP18.1, TP19.1, TP2.1, TP20.1, TP21.1, TP22.1, TP23.1, TP24.1, TP25.1, TP27.1, TP29.1, TP31.1, TP32.1, TP33.1, TP34.1, TP35.1, TP36.1, TP37.1, TP38.1, TP39.1, TP4.1, TP40.1, TP41.1, TP42.1, TP6.1, TP8.1, TP9.1
- net SWD.SWDIO: now reaches U1.13 (PA04)
- net SWD.SWDIO: now also U1.15 (PA06), U1.3 (PA02), U1.53 (PC02), U1.55 (PC04), U1.60 (PC06), TP26.1, TP28.1, TP3.1, TP30.1, TP5.1, TP7.1
Other:
- moved on the sheet: U1A

Commit message: stuff
Connections:
- net SWD.SWCLK: no longer TP1.1, TP2.1, TP20.1, TP21.1, U1.1 (PA00), U1.2 (PA01)
- new net: TP2.1, TP21.1, U1.2 (PA01)
- new net: TP1.1, TP20.1, U1.1 (PA00)
Changed lines of the file:
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@@
-		)
-	)
-	(label "SWD.SWCLK"
-		(at 196.85 76.2 0)
-		(effects
-			(font
-				(size 1.27 1.27)
-			)
-			(justify left bottom)
-		)
-	)
-	(label "SWD.SWCLK"
-		(at 196.85 78.74 0)
-		(effects
-			(font
-				(size 1.27 1.27)
-			)
-			(justify left bottom)
 		)
 	)
@@
 				)
 				(justify left)
+				(hide yes)
 			)
 		)
@@
 				)
 				(justify left)
-			)
-		)
+				(hide yes)
+			)
+		)

Commit message: stuff
Parts:
- added TP1, TP10, TP11, TP12, TP13, TP14, TP15, TP16, TP17, TP18, TP19, TP2, TP20, TP21, TP22, TP23, TP24, TP25, TP26, TP27, TP28, TP29, TP3, TP30, TP31, TP32, TP33, TP34, TP35, TP36, TP37, TP38, TP39, TP4, TP40, TP41, TP42, TP43, TP44, TP5, TP6, TP7, TP8, TP9: TestPoint, symbol Connector:TestPoint
Connections:
- net +3.3V: now also U1.21 (EXT), U1.26 (PB00), U1.27 (PB01), U1.28 (PB11), U1.31 (PB02), U1.32 (PB03), U1.36 (PB04), U1.37 (PB05), U1.39 (PB06), U1.47 (PB07), U1.49 (PB09), U1.50 (PB10); no longer U1.20 (VDDIO), U1.33 (VDDA), U1.34 (VDDIO), U1.42 (VDDIO), U1.44 (VDDREG), U1.56 (VDDIO), U1.62 (VDDREG), U1.69 (VDDIO), U1.7 (VDDIO), U1.79 (VCCAP3), U1.83 (VDDREG), U1.85 (VDDIO), U1.96 (VDDIO)
- net GND: now also U1.38 (PB13), U1.40 (PB14), U1.41 (PB15), U1.45 (PB16), U1.46 (PB17), U1.86 (PD00), U1.87 (PD01), U1.92 (PD05), U1.94 (PD07), U1.98 (PD09); no longer U1.101 (GND), U1.19 (GND), U1.30 (VSSA), U1.35 (GND), U1.43 (GND), U1.57 (GND), U1.6 (GND), U1.70 (GND), U1.80 (USBVSSA), U1.84 (VSSIO), U1.95 (GND)
- net SWD.SWCLK: now also U1.31 (PB02), TP7.1; no longer TP10.1, TP11.1, TP12.1, TP13.1, TP14.1, TP15.1, TP16.1, TP17.1, TP18.1, TP19.1, TP22.1, TP23.1, TP24.1, TP25.1, TP27.1, TP29.1, TP31.1, TP32.1, TP33.1, TP34.1, TP35.1, TP36.1, TP37.1, TP38.1, TP39.1, TP40.1, TP41.1, TP42.1, TP6.1, TP8.1, TP9.1, U1.10 (PA15), U1.11 (PA16), U1.12 (PA17), U1.14 (PA05), U1.16 (PA07), U1.17 (PA08), U1.18 (PA18), U1.22 (PA09), U1.23 (PA10), U1.24 (PA11), U1.25 (PA12), U1.51 (PC00), U1.52 (PC01), U1.54 (PC03), U1.58 (PC14), U1.59 (PC05), U1.61 (PC07), U1.63 (PC09), U1.64 (PC15), U1.65 (PC16), U1.66 (PC17), U1.67 (PC18), U1.68 (PC10), U1.71 (PC11), U1.72 (PC12), U1.73 (PC13), U1.74 (PC19), U1.8 (PA13), U1.9 (PA14)
- net SWD.SWDIO: now also U1.27 (PB01), TP6.1; no longer TP26.1, TP28.1, TP30.1, TP5.1, TP7.1, U1.13 (PA04), U1.15 (PA06), U1.53 (PC02), U1.55 (PC04), U1.60 (PC06)
- net ETH.RXDV: now reaches U1.100 (PD11)
- net ETH.RXDV: now also TP33.1, U1.68 (PC10), TP34.1
- net at U1.26 (PB00): now also TP4.1, TP5.1
- net ETH.MDIO: now reaches U1.28 (PB11)
- net ETH.MDIO: now also TP13.1, U1.25 (PA12), TP16.1
- net SPI5.MOSI: now reaches U1.29 (PB12)
- net SPI5.MOSI: now also TP14.1, U1.8 (PA13), TP17.1
- net SPI7.MOSI: now reaches U1.32 (PB03)
- net SPI7.MOSI: now also TP5.1, U1.13 (PA04), TP8.1
- net SPI7.MISO: now reaches U1.36 (PB04)
- net SPI7.MISO: now also TP6.1, U1.14 (PA05), TP9.1
- net SPI7.SCK: now reaches U1.37 (PB05)
- net SPI7.SCK: now also TP7.1, U1.15 (PA06), TP10.1
- net SPI5.MISO: now reaches U1.38 (PB13)
- net SPI5.MISO: now also TP15.1, U1.9 (PA14), TP18.1
- net SPI6.MOSI: now reaches U1.39 (PB06)
- net SPI6.MOSI: now also TP8.1, U1.16 (PA07), TP11.1
- net SPI5.SCK: now reaches U1.40 (PB14)
- net SPI5.SCK: now also TP16.1, U1.10 (PA15), TP19.1
- net SPI5.CS#: now reaches U1.41 (PB15)
- net SPI5.CS#: now also TP17.1, U1.11 (PA16), TP20.1
- net SPARE1: now reaches U1.45 (PB16)
- net SPARE1: now also TP18.1, U1.12 (PA17), TP21.1
- net SPARE2: now reaches U1.46 (PB17)
- net SPARE2: now also TP19.1, U1.18 (PA18), TP22.1
- net SPI6.MISO: now reaches U1.47 (PB07)
- net SPI6.MISO: now also TP9.1, U1.17 (PA08), TP12.1
- net SPI6.SCK: now reaches U1.48 (PB08)
- net SPI6.SCK: now also TP10.1, U1.22 (PA09), TP13.1
- net SPI6.CS#: now reaches U1.49 (PB09)
- net SPI6.CS#: now also TP11.1, U1.23 (PA10), TP14.1
- net ETH.MDC: now reaches U1.50 (PB10)
- net ETH.MDC: now also TP12.1, U1.24 (PA11), TP15.1
- net SPARE11: now reaches U1.75 (PC20)
- net SPARE11: now also TP1.1, TP44.1
- net SPI2.SCK: now reaches U1.76 (USB0PN)
- net SPI2.SCK: now also TP40.1, U1.66 (PC17), TP41.1
- net SPI2.CS#: now reaches U1.77 (USB0PP)
- net SPI2.CS#: now also TP41.1, U1.67 (PC18), TP42.1
- net SPI2.MISO: now reaches U1.78 (USB0ID)
- net SPI2.MISO: now also TP39.1, U1.65 (PC16), TP40.1
- net SPARE10: now reaches U1.82 (USRBIAS)
- net SPARE10: now also TP42.1, U1.74 (PC19), TP43.1
- net SPARE3: now reaches U1.86 (PD00)
- net SPARE3: now also TP22.1, TP23.1, U1.51 (PC00), TP23.1, TP24.1
- net SPARE4: now reaches U1.87 (PD01)
- net SPARE4: now also TP24.1, TP25.1, U1.52 (PC01), TP25.1, TP26.1
- net SPARE5: now reaches U1.88 (PD02)
- net SPARE5: now also TP26.1, U1.53 (PC02), TP27.1
- net ETH.TXD1: now reaches U1.89 (USB_DM)
- net ETH.TXD1: now also TP36.1, U1.73 (PC13), TP37.1
- net SPARE9: now reaches U1.90 (USB_DP)
- net SPARE9: now also TP37.1, U1.58 (PC14), TP38.1
- net ETH.TXEN: now reaches U1.91 (PD12)
- net ETH.TXEN: now also TP34.1, U1.71 (PC11), TP35.1
- net SPARE6: now reaches U1.92 (PD05)
- net SPARE6: now also TP27.1, U1.54 (PC03), TP28.1
- net SPARE7: now reaches U1.93 (PD06)
- net SPARE7: now also TP28.1, U1.55 (PC04), TP29.1
- net SPARE8: now reaches U1.94 (PD07)
- net SPARE8: now also TP29.1, U1.59 (PC05), TP30.1
- net ETH.RXD1: now reaches U1.97 (PD08)
- net ETH.RXD1: now also TP30.1, U1.60 (PC06), TP31.1
- net ETH.RXD0: now reaches U1.98 (PD09)
- net ETH.RXD0: now also TP31.1, U1.61 (PC07), TP32.1
- net ETH.RXER: now reaches U1.99 (PD10)
- net ETH.RXER: now also TP32.1, U1.63 (PC09), TP33.1
- new net: TP2.1, TP3.1
- new net ETH.TXD0: TP35.1, TP36.1, U1.72 (PC12)
- new net SPI2.MOSI: TP38.1, U1.64 (PC15)

Commit message: did alot of stuff
Parts:
- removed TP2, TP23, TP24, TP25 (x2), TP3, TP36, TP39: TestPoint, symbol Connector:TestPoint
- removed U1: PIC32CK1025GC01100-I/4SB, PIC32CK1025GC01100-I-4SB:TQFP100_4SB_6p3EP_MCH, symbol PIC32CK1025GC01100-I-4SB:PIC32CK1025GC01100-I_4SB
- added C1, C10, C11, C12, C14, C16, C2, C3, C4, C5, C6, C7, C8: 100n, Capacitor_SMD:C_0402_1005Metric, symbol Device:C
- added C13, C18, C9: 47u, Capacitor_SMD:C_1210_3225Metric, symbol Device:C
- added C15: 4.7u, Capacitor_SMD:C_0805_2012Metric, symbol Device:C
- added C17: 10u, Capacitor_SMD:C_0805_2012Metric, symbol Device:C
- added C19, C20, C21, C22: C, Capacitor_SMD:C_0402_1005Metric, symbol Device:C
- added D1, D2: LED, LED_SMD:LED_0805_2012Metric, symbol Device:LED
- added FB2: FerriteBead_Small, symbol Device:FerriteBead_Small
- added Q1, Q2: NMOS, symbol Simulation_SPICE:NMOS
- added R1, R2: 0, Resistor_SMD:R_0402_1005Metric, symbol Device:R
- added R3, R4: R, Resistor_SMD:R_0402_1005Metric, symbol Device:R
- added R5, R6, R8, R9: 10k, Resistor_SMD:R_0402_1005Metric, symbol Device:R
- added R7: 270, Resistor_SMD:R_0402_1005Metric, symbol Device:R
- added SW1: SW_Push, symbol Switch:SW_Push
- added TP43, TP45, TP46: TestPoint, symbol Connector:TestPoint
- added unit 2 of U1
- added Y1, Y2: Crystal, symbol Device:Crystal
- renumbered TP4 to TP47, TP5 to TP48, TP6 to TP49, TP7 to TP50, TP8 to TP51, TP9 to TP52, TP10 to TP53, TP11 to TP54, TP12 to TP55, TP13 to TP56, TP14 to TP57, TP15 to TP58, TP16 to TP59, TP17 to TP60, TP18 to TP61, TP19 to TP62, TP20 to TP63, TP21 to TP64, TP22 to TP65, TP23 to TP66, TP26 to TP67, TP27 to TP68, TP28 to TP69, TP29 to TP70, TP30 to TP71, TP31 to TP72, TP32 to TP73, TP33 to TP74, TP34 to TP75, TP35 to TP76, TP37 to TP77, TP38 to TP78, TP40 to TP79, TP41 to TP80, TP42 to TP81, TP1 to TP82, TP43 to TP83
Connections:
- net +3.3V: now also C1.1, C10.1, C11.1, C12.1, C13.1, C14.1, C15.1, C18.1, C2.1, C3.1, C4.1, C5.1, C6.1, C7.1, C8.1, C9.1, FB2.1, R3.1, R4.1, R5.1, R9.1, SW1.1, U1.20 (VDDIO), U1.34 (VDDIO), U1.42 (VDDIO), U1.44 (VDDREG), U1.56 (VDDIO), U1.62 (VDDREG), U1.69 (VDDIO), U1.7 (VDDIO), U1.79 (VCCAP3), U1.83 (VDDREG), U1.85 (VDDIO), U1.96 (VDDIO)
- net GND: now also C1.2, C10.2, C11.2, C12.2, C13.2, C14.2, C15.2, C16.2, C17.2, C18.2, C19.2, C2.2, C20.2, C21.2, C22.2, C3.2, C4.2, C5.2, C6.2, C7.2, C8.2, C9.2, D2.1 (K), Q1.3 (S), Q2.3 (S), R6.2, R7.2, R8.2, U1.101 (GND), U1.19 (GND), U1.30 (VSSA), U1.35 (GND), U1.43 (GND), U1.57 (GND), U1.6 (GND), U1.70 (GND), U1.80 (USBVSSA), U1.84 (VSSIO), U1.95 (GND)
- net SPARE1: no longer TP64.1, U1.45 (PB16)
- net SPARE10: no longer TP83.1, U1.82 (USRBIAS)
- net SPARE11: no longer TP44.1
- net SPARE2: no longer TP65.1, U1.46 (PB17)
- net SPARE4: no longer TP67.1, U1.87 (PD01)
- net SPARE5: no longer TP68.1, U1.88 (PD02)
- net SPARE6: no longer TP69.1, U1.92 (PD05)
- net SPARE7: no longer TP70.1, U1.93 (PD06)
- net SPARE8: no longer TP71.1, U1.94 (PD07)
- net SPARE9: no longer TP78.1, U1.90 (USB_DP)
- net SPI2.CS#: no longer TP81.1, U1.77 (USB0PP)
- net SPI2.MISO: no longer TP79.1, U1.78 (USB0ID)
- net SPI2.SCK: no longer TP80.1, U1.76 (USB0PN)
- net SPI5.CS#: no longer TP63.1, U1.41 (PB15)
- net SPI5.MISO: no longer TP61.1, U1.38 (PB13)
- net SPI5.MOSI: no longer TP60.1, U1.29 (PB12)
- net SPI5.SCK: no longer TP62.1, U1.40 (PB14)
- net SPI6.CS#: no longer TP57.1, U1.49 (PB09)
- net SPI6.MISO: no longer TP55.1, U1.47 (PB07)
- net SPI6.MOSI: no longer TP54.1, U1.39 (PB06)
- net SPI6.SCK: no longer TP56.1, U1.48 (PB08)
- net SPI7.MISO: now also TP5.1, U1.13 (PA04); no longer TP52.1, TP6.1, U1.14 (PA05), U1.36 (PB04)
- net SPI7.MOSI: now also R1.2; no longer TP5.1, TP51.1, U1.13 (PA04), U1.32 (PB03)
- net SPI7.SCK: now also TP6.1, U1.14 (PA05); no longer TP53.1, TP7.1, U1.15 (PA06), U1.37 (PB05)
- net SPARE12: now reaches TP47.1, TP48.1, U1.26 (PB00)
- net PA01: now reaches TP2.1, TP21.1, U1.2 (PA01)
- net PA01: now also R1.1, R2.1
- net JTAG.TDI: now reaches TP1.1, TP20.1, U1.1 (PA00)
- net EXT: now reaches U1.21 (EXT)
- net EXT: now also TP45.1, TP46.1
- net RESET#: now reaches U1.5 (RESET_N)
- net RESET#: now also TP44.1, Q2.1 (D), R5.2, TP43.1
- net ETH.MDC renamed SMI.MDC
- net SMI.MDC: no longer TP58.1, U1.50 (PB10)
- net ETH.MDIO renamed ADC_VINP10
- net ADC_VINP10: no longer TP13.1, U1.25 (PA12)
- net ETH.RXD0 renamed RMII.RXD0
- net RMII.RXD0: no longer TP73.1, U1.98 (PD09)
- net ETH.RXD1 renamed RMII.RXD1
- net RMII.RXD1: no longer TP72.1, U1.97 (PD08)
- net ETH.RXDV renamed RMII.CRSDV
- net RMII.CRSDV: no longer TP75.1, U1.100 (PD11)
- net ETH.RXER renamed RMII.RXER
- net RMII.RXER: no longer TP74.1, U1.99 (PD10)
- net ETH.TXD0 renamed RMII.TXD0
- net ETH.TXD1 renamed RMII.TXD1
- net RMII.TXD1: no longer TP77.1, U1.89 (USB_DM)
- net ETH.TXEN renamed RMII.TXEN
- net RMII.TXEN: no longer TP76.1, U1.91 (PD12)
- net SPARE3 renamed RMII.REFCK
- net RMII.REFCK: no longer TP66.1, U1.86 (PD00)
- net SWD.SWCLK renamed JTAG.TCK
- net JTAG.TCK: no longer TP50.1, U1.31 (PB02)
- net SWD.SWDIO renamed JTAG.TMS
- net JTAG.TMS: no longer TP49.1, U1.27 (PB01)
- new net: C16.1, C17.1, FB2.2, U1.33 (VDDA)
- new net: D1.2 (A), R3.2
- new net: D1.1 (K), Q1.1 (D)
- new net: D2.2 (A), R4.2
- new net ADC_VINP11: TP60.1, U1.29 (PB12)
- new net JTAG.TDO: R2.2
- new net RST_BTN: Q2.2 (G), R6.1, SW1.2
- new net SDMMC0_SDCD: TP76.1, U1.91 (PD12)
- new net SDMMC0_SDCK: TP74.1, U1.99 (PD10)
- new net SDMMC0_SDCMD: TP70.1, U1.93 (PD06)
- new net SDMMC0_SDDAT0: TP71.1, U1.94 (PD07)
- new net SDMMC0_SDDAT1: TP75.1, U1.100 (PD11)
- new net SDMMC0_SDDAT2: TP72.1, U1.97 (PD08)
- new net SDMMC0_SDDAT3: TP73.1, U1.98 (PD09)
- new net SDMMC0_SDWP: TP69.1, U1.92 (PD05)
- new net SMI.MDIO: TP13.1, U1.25 (PA12)
- new net SPARE13: TP49.1, U1.27 (PB01)
- new net SPARE14: TP57.1, U1.49 (PB09)
- new net SPARE15: TP58.1, U1.50 (PB10)
- new net SPARE16: TP62.1, U1.40 (PB14)
- new net SPARE17: TP63.1, U1.41 (PB15)
- new net SPI3.CS#: TP56.1, U1.48 (PB08)
- new net SPI3.MISO: TP65.1, U1.46 (PB17)
- new net SPI3.MOSI: TP64.1, U1.45 (PB16)
- new net SPI3.SCK: TP55.1, U1.47 (PB07)
- new net SPI4.CS#: TP54.1, U1.39 (PB06)
- new net SPI4.MISO: TP53.1, U1.37 (PB05)
- new net SPI4.MOSI: TP52.1, U1.36 (PB04)
- new net SPI4.SCK: TP61.1, U1.38 (PB13)
- new net SPI7.CS#: TP7.1, U1.15 (PA06)
- new net STATUS_LED: Q1.2 (G)
- new net TSUCOMP: TP68.1, U1.88 (PD02)
- new net USB0ID: R8.1, R9.2, TP79.1, U1.78 (USB0ID)
- new net USB_FS.D+: TP78.1, U1.90 (USB_DP)
- new net USB_FS.D-: TP77.1, U1.89 (USB_DM)
- new net USB_HS.D+: TP81.1, U1.77 (USB0PP)
- new net USB_HS.D-: TP80.1, U1.76 (USB0PN)
- new net USRBIAS: R7.1, TP83.1, U1.82 (USRBIAS)
- new net XIN: C19.1, TP66.1, U1.86 (PD00), Y1.1
- new net XIN32: C22.1, TP50.1, U1.31 (PB02), Y2.1
- new net XOUT: C21.1, TP67.1, U1.87 (PD01), Y1.2
- new net XOUT32: C20.1, TP51.1, U1.32 (PB03), Y2.2
Other:
- note added: "DNM"
- note added: "Design Note: 24 KHz 8pF 10ppm Crystal"
- note added: "Design Note: 32.768 KHz 10pF 10ppm Crystal"
- note added: "Design Note: Force USB OTG to Device role"
- note added: "Design Note: TSUCOMP compares PTP time to value option to trigger ADC perhaps"
- note added: "Microcontroller"
- moved on the sheet: TP1, TP10, TP11, TP12, TP13, TP14, TP15, TP16, TP17, TP18, TP19, TP2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

Commit message: stuff
Parts:
- removed R1: 0, Resistor_SMD:R_0402_1005Metric, symbol Device:R
- added R56, R57, R58, R59: 27, Resistor_SMD:R_0402_1005Metric, symbol Device:R
Connections:
- net USB_FS.D+: now also R57.2
- net USB_FS.D-: now also R56.2
- net USB_HS.D+: now also R59.2
- net USB_HS.D-: now also R58.2
- net SDMMC0_SDCD renamed SDMMC0.SDCD
- net SDMMC0_SDCK renamed SDMMC0.SDCK
- net SDMMC0_SDCMD renamed SDMMC0.SDCMD
- net SDMMC0_SDDAT0 renamed SDMMC0.SDDAT0
- net SDMMC0_SDDAT1 renamed SDMMC0.SDDAT1
- net SDMMC0_SDDAT2 renamed SDMMC0.SDDAT2
- net SDMMC0_SDDAT3 renamed SDMMC0.SDDAT3
- net SDMMC0_SDWP renamed SDMMC0.SDWP
- net SPI4.CS# renamed NC_SERCOM4_PAD3
- net SPI4.MISO renamed UART4.RX
- net SPI4.MOSI renamed UART4.TX
- net SPI4.SCK renamed NC_SERCOM4_PAD2
- net SPI7.CS# renamed NC_SERCOM7_PAD3
- net SPI7.MISO renamed I2C7.SDA
- net SPI7.SCK renamed I2C7.SCL
- new net USB.D+: R57.1, R59.1
- new net USB.D-: R56.1, R58.1
Other:
- note added: "CAD Note: Place without stubs"
- moved on the sheet: R2, R7

Commit message: started on adc
Other:
- moved on the sheet: C10, C12, C4, C6, C7, C8
Changed lines of the file:
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@@
 	(symbol
 		(lib_id "Device:C")
-		(at 347.98 140.97 0)
+		(at 332.74 140.97 0)
 		(unit 1)
 		(exclude_from_sim no)
@@
 		(dnp no)
 		(property "Reference" "C12"
-			(at 348.996 138.176 0)
+			(at 333.756 138.176 0)
 			(effects
 				(font
@@
 		)
 		(property "Value" "100n"
-			(at 348.996 143.51 0)
+			(at 333.756 143.51 0)
 			(effects
 				(font
@@
 		)
 		(property "Footprint" "Capacitor_SMD:C_0402_1005Metric"
-			(at 348.9452 144.78 0)
+			(at 333.7052 144.78 0)
 			(effects
 				(font
@@
 		)
 		(property "Datasheet" "~"
-			(at 347.98 140.97 0)
+			(at 332.74 140.97 0)
 			(effects
 				(font
@@
 		)
 		(property "Description" "Unpolarized capacitor"
-			(at 347.98 140.97 0)
+			(at 332.74 140.97 0)
 			(effects
 				(font
@@
 	(symbol
 		(lib_id "Device:C")
-		(at 332.74 140.97 0)
+		(at 347.98 140.97 0)
 		(unit 1)
 		(exclude_from_sim no)
@@
 		(dnp no)
 		(property "Reference" "C10"
-			(at 333.756 138.176 0)
+			(at 348.996 138.176 0)
 			(effects
 				(font
@@
 		)
 		(property "Value" "100n"
-			(at 333.756 143.51 0)
+			(at 348.996 143.51 0)
 			(effects
 				(font
@@
 		)
 		(property "Footprint" "Capacitor_SMD:C_0402_1005Metric"
-			(at 333.7052 144.78 0)
+			(at 348.9452 144.78 0)
 			(effects
 				(font
@@
 		)
 		(property "Datasheet" "~"
-			(at 332.74 140.97 0)
+			(at 347.98 140.97 0)
 			(effects
 				(font
@@
 		)
 		(property "Description" "Unpolarized capacitor"
-			(at 332.74 140.97 0)
+			(at 347.98 140.97 0)
 			(effects
 				(font
@@
 	(symbol
 		(lib_id "Device:C")
-		(at 309.88 121.92 0)
+		(at 325.12 121.92 0)
 		(unit 1)
 		(exclude_from_sim no)
@@
 		(dnp no)
 		(property "Reference" "C4"
-			(at 310.896 119.126 0)
+			(at 326.136 119.126 0)
 			(effects
 				(font
@@
 		)
 		(property "Value" "100n"
-			(at 310.896 124.46 0)
+			(at 326.136 124.46 0)
 			(effects
 				(font
@@
 		)
 		(property "Footprint" "Capacitor_SMD:C_0402_1005Metric"
-			(at 310.8452 125.73 0)
+			(at 326.0852 125.73 0)
 			(effects
 				(font
@@
 		)
 		(property "Datasheet" "~"
-			(at 309.88 121.92 0)
+			(at 325.12 121.92 0)
 			(effects
 				(font
@@
 		)
 		(property "Description" "Unpolarized capacitor"
-			(at 309.88 121.92 0)
+			(at 325.12 121.92 0)
 			(effects
 				(font
@@
 	(symbol
 		(lib_id "Device:C")
-		(at 325.12 121.92 0)
+		(at 309.88 121.92 0)
 		(unit 1)
 		(exclude_from_sim no)
@@
 		(dnp no)
 		(property "Reference" "C6"
-			(at 326.136 119.126 0)
+			(at 310.896 119.126 0)
 			(effects
 				(font
@@
 		)
 		(property "Value" "100n"
-			(at 326.136 124.46 0)
+			(at 310.896 124.46 0)
 			(effects
 				(font
@@
 		)
 		(property "Footprint" "Capacitor_SMD:C_0402_1005Metric"
-			(at 326.0852 125.73 0)
+			(at 310.8452 125.73 0)
 			(effects
 				(font
@@
 		)
 		(property "Datasheet" "~"
-			(at 325.12 121.92 0)
+			(at 309.88 121.92 0)
 			(effects
 				(font
@@
 		)
 		(property "Description" "Unpolarized capacitor"
-			(at 325.12 121.92 0)
+			(at 309.88 121.92 0)
 			(effects
 				(font
@@
 	(symbol
 		(lib_id "Device:C")
-		(at 294.64 121.92 0)
+		(at 302.26 121.92 0)
 		(unit 1)
 		(exclude_from_sim no)
@@
 		(dnp no)
 		(property "Reference" "C7"
-			(at 295.656 119.126 0)
+			(at 303.276 119.126 0)
 			(effects
 				(font
@@
 		)
 		(property "Value" "100n"
-			(at 295.656 124.46 0)
+			(at 303.276 124.46 0)
 			(effects
 				(font
@@
 		)
 		(property "Footprint" "Capacitor_SMD:C_0402_1005Metric"
-			(at 295.6052 125.73 0)
+			(at 303.2252 125.73 0)
 			(effects
 				(font
@@
 		)
 		(property "Datasheet" "~"
-			(at 294.64 121.92 0)
+			(at 302.26 121.92 0)
 			(effects
 				(font
@@
 		)
 		(property "Description" "Unpolarized capacitor"
-			(at 294.64 121.92 0)
+			(at 302.26 121.92 0)
 			(effects
 				(font
@@
 	(symbol
 		(lib_id "Device:C")
-		(at 302.26 121.92 0)
+		(at 294.64 121.92 0)
 		(unit 1)
 		(exclude_from_sim no)
@@
 		(dnp no)
 		(property "Reference" "C8"
-			(at 303.276 119.126 0)
+			(at 295.656 119.126 0)
 			(effects
 				(font
@@
 		)
 		(property "Value" "100n"
-			(at 303.276 124.46 0)
+			(at 295.656 124.46 0)
 			(effects
 				(font
@@
 		)
 		(property "Footprint" "Capacitor_SMD:C_0402_1005Metric"
-			(at 303.2252 125.73 0)
+			(at 295.6052 125.73 0)
 			(effects
 				(font
@@
 		)
 		(property "Datasheet" "~"
-			(at 302.26 121.92 0)
+			(at 294.64 121.92 0)
 			(effects
 				(font
@@
 		)
 		(property "Description" "Unpolarized capacitor"
-			(at 302.26 121.92 0)
+			(at 294.64 121.92 0)
 			(effects
 				(font

Commit message: did stuff
Parts:
- renumbered C15 to C1, C5 to C10, C4 to C11, C3 to C12, C2 to C13, C1 to C14, C13 to C15, C12 to C16, C11 to C17, C10 to C18, C21 to C19, C14 to C2, C19 to C20, C20 to C21, C18 to C3, C17 to C4, C16 to C5, C9 to C6, C8 to C7, C7 to C8, C6 to C9, FB2 to FB1, R5 to R1, R3 to R10, R4 to R11, R6 to R12, R56 to R3, R57 to R4, R58 to R5, R59 to R6, R9 to R7, R7 to R8, R8 to R9, TP43 to TP1, TP47 to TP10, TP48 to TP11, TP4 to TP12, TP49 to TP13, TP5 to TP14, TP50 to TP15, TP6 to TP16, TP51 to TP17, TP7 to TP18, TP52 to TP19, TP44 to TP2, TP8 to TP20, TP53 to TP21, TP9 to TP22, TP54 to TP23, TP10 to TP24, TP55 to TP25, TP11 to TP26, TP56 to TP27, TP12 to TP28, TP57 to TP29, TP1 to TP3, TP13 to TP30, TP58 to TP31, TP14 to TP32, TP59 to TP33, TP15 to TP34, TP60 to TP35, TP16 to TP36, TP61 to TP37, TP17 to TP38, TP62 to TP39, TP20 to TP4, TP18 to TP40, TP63 to TP41, TP19 to TP42, TP64 to TP43, TP65 to TP44, TP22 to TP45, TP24 to TP46, TP66 to TP47, TP26 to TP48, TP67 to TP49, TP45 to TP5, TP27 to TP50, TP68 to TP51, TP28 to TP52, TP69 to TP53, TP29 to TP54, TP70 to TP55, TP30 to TP56, TP71 to TP57, TP31 to TP58, TP72 to TP59, TP46 to TP6, TP32 to TP60, TP73 to TP61, TP33 to TP62, TP74 to TP63, TP34 to TP64, TP75 to TP65, TP35 to TP66, TP76 to TP67, TP36 to TP68, TP37 to TP69, TP2 to TP7, TP77 to TP70, TP38 to TP71, TP78 to TP72, TP39 to TP73, TP40 to TP74, TP79 to TP75, TP41 to TP76, TP80 to TP77, TP42 to TP78, TP81 to TP79, TP21 to TP8, TP82 to TP80, TP83 to TP81, TP3 to TP9
