File: mcu.kicad_sch (KiCad schematic)
At the start: 128 parts, among them Q3 BSS138LT1G, Q4 BSS138LT1G, Q5 BSS138LT1G, Q6 BSS138LT1G, SW1 TS110926043, SW2 TS110926043, U1 PIC32CK1025GC01100-I/4SB, X2 Q13FC1350000400, X3 X322512MSB4SI

Commit message: did stuff, amongst others changed to op-amp input filter
Parts:
- SW1, SW2: LCSC (none) -> C22375349
- X2: LCSC (none) -> C32346
- X3: LCSC (none) -> C9002

Commit message: fixed a bunch of errors, set pin type on alot of pins
Parts:
- added C269: 100n 50V, Capacitor_SMD:C_0402_1005Metric, symbol Device:C
- R3, R4: now not fitted
Connections:
- net SPARE11 is gone; now on net ETH_RST#: TP80.1, U1.75 (PC20)
- net GND: now also C269.2
- net +5V_USB: now reaches U1.81 (VBUS)
- net +5V_USB: now also C269.1
- net PA01 renamed INT_JTAG_TDO
Other:
- moved on the sheet: R2
