File: netdaq.kicad_sch (KiCad schematic)
At the start: 0 parts

Commit message: did alot of stuff
Other:
- added sheet Ethernet Connector (eth_conn.kicad_sch)
- added sheet Ethernet PHY (eth_phy.kicad_sch)
- sheet MCU ports: added ETH_RST#, RESET#, RMII{RMII}, SDMMC0{MMC}, SMI{SMI}, SPI2{SPI}, SPI3{SPI}, SPI4{SPI}, SPI5{SPI}, SPI6{SPI}, SPI7{SPI}, TSUCOMP, USB_FS{USB}, USB_HS{USB}, {JTAG}; removed none

Commit message: did stuff
Other:
- added sheet DAQ Connector (daq_conn.kicad_sch)
- added sheet PoE Regulator (poe_reg.kicad_sch)
Changed lines of the file:
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@@
+	)
+	(sheet
+		(at 156.21 104.14)
+		(size 21.59 19.05)
+		(exclude_from_sim no)
+		(in_bom yes)
+		(on_board yes)
+		(dnp no)
+		(fields_autoplaced yes)
+		(stroke
+			(width 0.1524)
+			(type solid)
+		)
+		(fill
+			(color 0 0 0 0.0000)
+		)
+		(property "Sheetname" "PoE Regulator"
+			(at 156.21 103.4284 0)
+			(effects
+				(font
+					(size 1.27 1.27)
+				)
+				(justify left bottom)
+			)
+		)
+		(property "Sheetfile" "poe_reg.kicad_sch"
+			(at 156.21 123.7746 0)
+			(effects
+				(font
+					(size 1.27 1.27)
+				)
+				(justify left top)
+			)
+		)
+		(instances
+			(project "netdaq"
+				(path "/2970f661-65ab-4e2b-aeda-d76d1044f2b8"
+					(page "6")
+				)
+			)
+		)
+	)
+	(sheet
+		(at 241.3 146.05)
+		(size 29.21 25.4)
+		(exclude_from_sim no)
+		(in_bom yes)
+		(on_board yes)
+		(dnp no)
+		(fields_autoplaced yes)
+		(stroke
+			(width 0.1524)
+			(type solid)
+		)
+		(fill
+			(color 0 0 0 0.0000)
+		)
+		(property "Sheetname" "DAQ Connector"
+			(at 241.3 145.3384 0)
+			(effects
+				(font
+					(size 1.27 1.27)
+				)
+				(justify left bottom)
+			)
+		)
+		(property "Sheetfile" "daq_conn.kicad_sch"
+			(at 241.3 172.0346 0)
+			(effects
+				(font
+					(size 1.27 1.27)
+				)
+				(justify left top)
+			)
+		)
+		(instances
+			(project "netdaq"
+				(path "/2970f661-65ab-4e2b-aeda-d76d1044f2b8"
+					(page "5")
+				)
+			)
+		)
 	)
 	(sheet

Commit message: did stuff
Other:
- added sheet PD Controller (pd_ctrl.kicad_sch)
Changed lines of the file:
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@@
+	)
+	(sheet
+		(at 156.21 133.35)
+		(size 21.59 17.78)
+		(exclude_from_sim no)
+		(in_bom yes)
+		(on_board yes)
+		(dnp no)
+		(fields_autoplaced yes)
+		(stroke
+			(width 0.1524)
+			(type solid)
+		)
+		(fill
+			(color 0 0 0 0.0000)
+		)
+		(property "Sheetname" "PD Controller"
+			(at 156.21 132.6384 0)
+			(effects
+				(font
+					(size 1.27 1.27)
+				)
+				(justify left bottom)
+			)
+		)
+		(property "Sheetfile" "pd_ctrl.kicad_sch"
+			(at 156.21 151.7146 0)
+			(effects
+				(font
+					(size 1.27 1.27)
+				)
+				(justify left top)
+			)
+		)
+		(instances
+			(project "netdaq"
+				(path "/2970f661-65ab-4e2b-aeda-d76d1044f2b8"
+					(page "7")
+				)
+			)
+		)
 	)
 	(sheet

Commit message: stuff
Other:
- added sheet 3V3 Regulator (3v3_reg.kicad_sch)
- added sheet Debug Connector (debug_conn.kicad_sch)
- added sheet USB Connector (usb_conn.kicad_sch)
Changed lines of the file:
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@@
+	)
+	(sheet
+		(at 307.34 154.94)
+		(size 22.86 20.32)
+		(exclude_from_sim no)
+		(in_bom yes)
+		(on_board yes)
+		(dnp no)
+		(fields_autoplaced yes)
+		(stroke
+			(width 0.1524)
+			(type solid)
+		)
+		(fill
+			(color 0 0 0 0.0000)
+		)
+		(property "Sheetname" "Debug Connector"
+			(at 307.34 154.2284 0)
+			(effects
+				(font
+					(size 1.27 1.27)
+				)
+				(justify left bottom)
+			)
+		)
+		(property "Sheetfile" "debug_conn.kicad_sch"
+			(at 307.34 175.8446 0)
+			(effects
+				(font
+					(size 1.27 1.27)
+				)
+				(justify left top)
+			)
+		)
+		(instances
+			(project "netdaq"
+				(path "/2970f661-65ab-4e2b-aeda-d76d1044f2b8"
+					(page "9")
+				)
+			)
+		)
 	)
 	(sheet
@@
 	)
 	(sheet
-		(at 241.3 146.05)
+		(at 129.54 133.35)
+		(size 19.05 17.78)
+		(exclude_from_sim no)
+		(in_bom yes)
+		(on_board yes)
+		(dnp no)
+		(fields_autoplaced yes)
+		(stroke
+			(width 0.1524)
+			(type solid)
+		)
+		(fill
+			(color 0 0 0 0.0000)
+		)
+		(property "Sheetname" "3V3 Regulator"
+			(at 129.54 132.6384 0)
+			(effects
+				(font
+					(size 1.27 1.27)
+				)
+				(justify left bottom)
+			)
+		)
+		(property "Sheetfile" "3v3_reg.kicad_sch"
+			(at 129.54 151.7146 0)
+			(effects
+				(font
+					(size 1.27 1.27)
+				)
+				(justify left top)
+			)
+		)
+		(instances
+			(project "netdaq"
+				(path "/2970f661-65ab-4e2b-aeda-d76d1044f2b8"
+					(page "10")
+				)
+			)
+		)
+	)
+	(sheet
+		(at 195.58 242.57)
 		(size 29.21 25.4)
 		(exclude_from_sim no)
@@
 		)
 		(property "Sheetname" "DAQ Connector"
-			(at 241.3 145.3384 0)
+			(at 195.58 241.8584 0)
 			(effects
 				(font
@@
 		)
 		(property "Sheetfile" "daq_conn.kicad_sch"
-			(at 241.3 172.0346 0)
+			(at 195.58 268.5546 0)
 			(effects
 				(font
@@
 				(path "/2970f661-65ab-4e2b-aeda-d76d1044f2b8"
 					(page "5")
+				)
+			)
+		)
+	)
+	(sheet
+		(at 128.27 74.93)
+		(size 20.32 19.05)
+		(exclude_from_sim no)
+		(in_bom yes)
+		(on_board yes)
+		(dnp no)
+		(stroke
+			(width 0.1524)
+			(type solid)
+		)
+		(fill
+			(color 0 0 0 0.0000)
+		)
+		(property "Sheetname" "USB Connector"
+			(at 127.762 72.39 0)
+			(effects
+				(font
+					(size 1.27 1.27)
+				)
+				(justify left bottom)
+			)
+		)
+		(property "Sheetfile" "usb_conn.kicad_sch"
+			(at 127.762 73.152 0)
+			(effects
+				(font
+					(size 1.27 1.27)
+				)
+				(justify left top)
+			)
+		)
+		(pin "USB{USB}" bidirectional
+			(at 138.43 93.98 270)
+			(effects
+				(font
+					(size 1.27 1.27)
+				)
+				(justify left)
+			)
+		)
+		(instances
+			(project "netdaq"
+				(path "/2970f661-65ab-4e2b-aeda-d76d1044f2b8"
+					(page "8")
 				)
 			)
@@
 		(on_board yes)
 		(dnp no)
-		(fields_autoplaced yes)
 		(stroke
 			(width 0.1524)
@@
 		)
 		(property "Sheetname" "MCU"
-			(at 189.23 145.3384 0)
+			(at 186.944 143.51 0)
 			(effects
 				(font
@@
 		)
 		(property "Sheetfile" "mcu.kicad_sch"
-			(at 189.23 179.6546 0)
-			(effects
-				(font
+			(at 186.944 144.018 0)
+			(effects
+				(font

Commit message: stuff
Other:
- added sheet SDMMC (sdmmc.kicad_sch)
- sheet Debug Connector ports: added UART{UART}; removed none
- sheet Ethernet Connector ports: added POE_V+, POE_V-; removed none
- sheet MCU ports: added I2C7{I2C}, UART4{UART}; removed SPI4{SPI}, SPI7{SPI}
Changed lines of the file:
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@@
+	(bus
+		(pts
+			(xy 118.11 93.98) (xy 118.11 161.29)
+		)
+		(stroke
+			(width 0)
+			(type default)
+		)
+	)
+	(bus
+		(pts
+			(xy 228.6 163.83) (xy 299.72 163.83)
+		)
+		(stroke
+			(width 0)
+			(type default)
+		)
+	)
 	(bus
 		(pts
@@
 	(bus
 		(pts
+			(xy 228.6 151.13) (xy 265.43 151.13)
+		)
+		(stroke
+			(width 0)
+			(type default)
+		)
+	)
+	(bus
+		(pts
+			(xy 118.11 161.29) (xy 189.23 161.29)
+		)
+		(stroke
+			(width 0)
+			(type default)
+		)
+	)
+	(bus
+		(pts
 			(xy 212.09 93.98) (xy 212.09 146.05)
 		)
@@
 			(width 0)
 			(type default)
+		)
+	)
+	(label "USB{USB}"
+		(at 176.53 161.29 0)
+		(effects
+			(font
+				(size 1.27 1.27)
+			)
+			(justify left bottom)
 		)
 	)
@@
 		)
 	)
+	(label "SDMMC{MMC}"
+		(at 236.22 151.13 0)
+		(effects
+			(font
+				(size 1.27 1.27)
+			)
+			(justify left bottom)
+		)
+	)
 	(label "MDI{MDI}"
 		(at 185.42 80.01 0)
@@
 		)
 	)
+	(label "DBG_UART{UART}"
+		(at 236.22 163.83 0)
+		(effects
+			(font
+				(size 1.27 1.27)
+			)
+			(justify left bottom)
+		)
+	)
 	(sheet
 		(at 199.39 74.93)
@@
 	)
 	(sheet
-		(at 307.34 154.94)
+		(at 265.43 147.32)
+		(size 19.05 7.62)
+		(exclude_from_sim no)
+		(in_bom yes)
+		(on_board yes)
+		(dnp no)
+		(fields_autoplaced yes)
+		(stroke
+			(width 0.1524)
+			(type solid)
+		)
+		(fill
+			(color 0 0 0 0.0000)
+		)
+		(property "Sheetname" "SDMMC"
+			(at 265.43 146.6084 0)
+			(effects
+				(font
+					(size 1.27 1.27)
+				)
+				(justify left bottom)
+			)
+		)
+		(property "Sheetfile" "sdmmc.kicad_sch"
+			(at 265.43 155.5246 0)
+			(effects
+				(font
+					(size 1.27 1.27)
+				)
+				(justify left top)
+			)
+		)
+		(property "Field2" ""
+			(at 265.43 147.32 0)
+			(effects
+				(font
+					(size 1.27 1.27)
+				)
+			)
+		)
+		(pin "MMC{MMC}" bidirectional
+			(at 265.43 151.13 180)
+			(effects
+				(font
+					(size 1.27 1.27)
+				)
+				(justify left)
+			)
+		)
+		(instances
+			(project "netdaq"
+				(path "/2970f661-65ab-4e2b-aeda-d76d1044f2b8"
+					(page "11")
+				)
+			)
+		)
+	)
+	(sheet
+		(at 299.72 156.21)
 		(size 22.86 20.32)
 		(exclude_from_sim no)
@@
 		)
 		(property "Sheetname" "Debug Connector"
-			(at 307.34 154.2284 0)
+			(at 299.72 155.4984 0)
 			(effects
 				(font
@@
 		)
 		(property "Sheetfile" "debug_conn.kicad_sch"
-			(at 307.34 175.8446 0)
-			(effects
-				(font
-					(size 1.27 1.27)
-				)
-				(justify left top)
+			(at 299.72 177.1146 0)
+			(effects
+				(font
+					(size 1.27 1.27)
+				)
+				(justify left top)
+			)
+		)
+		(pin "UART{UART}" bidirectional
+			(at 299.72 163.83 180)
+			(effects
+				(font
+					(size 1.27 1.27)
+				)
+				(justify left)
 			)
 		)
@@
 	)
 	(sheet
-		(at 128.27 74.93)
+		(at 107.95 74.93)
 		(size 20.32 19.05)
 		(exclude_from_sim no)
@@
 		)
 		(property "Sheetname" "USB Connector"
-			(at 127.762 72.39 0)
+			(at 107.442 72.39 0)
 			(effects
 				(font
@@
 		)
 		(property "Sheetfile" "usb_conn.kicad_sch"
-			(at 127.762 73.152 0)
+			(at 107.442 73.152 0)
 			(effects
 				(font
@@
 		)
 		(pin "USB{USB}" bidirectional
-			(at 138.43 93.98 270)
+			(at 118.11 93.98 270)
 			(effects
 				(font
@@
 		)
 		(pin "SPI2{SPI}" bidirectional
-			(at 189.23 151.13 180)
+			(at 204.47 179.07 270)
 			(effects
 				(font
@@
 		)
 		(pin "SPI3{SPI}" bidirectional
-			(at 189.23 153.67 180)
-			(effects
-				(font
-					(size 1.27 1.27)
-				)
-				(justify left)
-			)
-		)
-		(pin "SPI4{SPI}" bidirectional
-			(at 189.23 156.21 180)
+			(at 207.01 179.07 270)
 			(effects
 				(font
@@
 		)
 		(pin "SPI5{SPI}" bidirectional
-			(at 189.23 158.75 180)
+			(at 209.55 179.07 270)
 			(effects
 				(font
@@
 		)
 		(pin "SPI6{SPI}" bidirectional
-			(at 189.23 161.29 180)
-			(effects
-				(font
-					(size 1.27 1.27)
-				)
-				(justify left)
-			)
-		)
-		(pin "SPI7{SPI}" bidirectional
-			(at 189.23 163.83 180)
+			(at 212.09 179.07 270)
 			(effects
 				(font
@@
 		)
 		(pin "{JTAG}" bidirectional
-			(at 228.6 154.94 0)
+			(at 228.6 166.37 0)
 			(effects
 				(font
@@
 		)
 		(pin "USB_FS{USB}" bidirectional
-			(at 228.6 171.45 0)
-			(effects
-				(font
-					(size 1.27 1.27)
-				)
-				(justify right)
+			(at 189.23 163.83 180)
+			(effects
+				(font
+					(size 1.27 1.27)
+				)
+				(justify left)
 			)
 		)
 		(pin "USB_HS{USB}" bidirectional
-			(at 228.6 168.91 0)
-			(effects
-				(font
-					(size 1.27 1.27)
-				)
-				(justify right)
+			(at 189.23 161.29 180)
+			(effects
+				(font
+					(size 1.27 1.27)
+				)
+				(justify left)
 			)
 		)
@@
 			)
 		)
+		(pin "I2C7{I2C}" bidirectional
+			(at 228.6 157.48 0)
+			(effects
+				(font
+					(size 1.27 1.27)
+				)
+				(justify right)
+			)
+		)
+		(pin "UART4{UART}" bidirectional
+			(at 228.6 163.83 0)
+			(effects
+				(font
+					(size 1.27 1.27)
+				)
+				(justify right)
+			)
+		)
 		(instances
 			(project "netdaq"
@@
 			)
 		)
+		(pin "POE_V+" output
+			(at 163.83 93.98 270)
+			(effects
+				(font
+					(size 1.27 1.27)
+				)
+				(justify left)
+			)
+		)
+		(pin "POE_V-" output
+			(at 166.37 93.98 270)
+			(effects
+				(font
+					(size 1.27 1.27)
+				)
+				(justify left)
+			)
+		)

Commit message: started on adc
Other:
- added sheet ADC Filter (adc_filt.kicad_sch)
- added sheet ADC1 (adc.kicad_sch)
- added sheet ADC2 (adc.kicad_sch)
- added sheet ADC3 (adc.kicad_sch)
- added sheet ADC4 (adc.kicad_sch)

Commit message: did stuff
Other:
- sheet DAQ Connector ports: added ADC[1..8], ADC[17..24], ADC[24..32], ADC[9..16]; removed none
Changed lines of the file:
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@@
+	(bus
+		(pts
+			(xy 215.9 236.22) (xy 254 236.22)
+		)
+		(stroke
+			(width 0)
+			(type default)
+		)
+	)
 	(bus
 		(pts
@@
 	(bus
 		(pts
+			(xy 208.28 233.68) (xy 198.12 233.68)
+		)
+		(stroke
+			(width 0)
+			(type default)
+		)
+	)
+	(bus
+		(pts
+			(xy 208.28 242.57) (xy 208.28 233.68)
+		)
+		(stroke
+			(width 0)
+			(type default)
+		)
+	)
+	(bus
+		(pts
 			(xy 226.06 161.29) (xy 226.06 194.31)
 		)
@@
 		)
 	)
+	(bus
+		(pts
+			(xy 198.12 215.9) (xy 198.12 233.68)
+		)
+		(stroke
+			(width 0)
+			(type default)
+		)
+	)
 	(wire
 		(pts
@@
 	(bus
 		(pts
+			(xy 212.09 233.68) (xy 226.06 233.68)
+		)
+		(stroke
+			(width 0)
+			(type default)
+		)
+	)
+	(bus
+		(pts
 			(xy 121.92 45.72) (xy 121.92 113.03)
 		)
@@
 	(bus
 		(pts
+			(xy 254 215.9) (xy 254 236.22)
+		)
+		(stroke
+			(width 0)
+			(type default)
+		)
+	)
+	(bus
+		(pts
+			(xy 204.47 242.57) (xy 204.47 236.22)
+		)
+		(stroke
+			(width 0)
+			(type default)
+		)
+	)
+	(bus
+		(pts
 			(xy 215.9 130.81) (xy 215.9 152.4)
 		)
@@
 	(bus
 		(pts
+			(xy 212.09 242.57) (xy 212.09 233.68)
+		)
+		(stroke
+			(width 0)
+			(type default)
+		)
+	)
+	(bus
+		(pts
 			(xy 170.18 152.4) (xy 170.18 194.31)
 		)
@@
 	(bus
 		(pts
+			(xy 170.18 215.9) (xy 170.18 236.22)
+		)
+		(stroke
+			(width 0)
+			(type default)
+		)
+	)
+	(bus
+		(pts
 			(xy 215.9 45.72) (xy 215.9 97.79)
 		)
@@
 	(bus
 		(pts
+			(xy 204.47 236.22) (xy 170.18 236.22)
+		)
+		(stroke
+			(width 0)
+			(type default)
+		)
+	)
+	(bus
+		(pts
+			(xy 226.06 215.9) (xy 226.06 233.68)
+		)
+		(stroke
+			(width 0)
+			(type default)
+		)
+	)
+	(bus
+		(pts
+			(xy 215.9 242.57) (xy 215.9 236.22)
+		)
+		(stroke
+			(width 0)
+			(type default)
+		)
+	)
+	(bus
+		(pts
 			(xy 213.36 161.29) (xy 226.06 161.29)
 		)
@@
 			(width 0)
 			(type default)
+		)
+	)
+	(label "GPIO[25..32]"
+		(at 254 228.6 90)
+		(effects
+			(font
+				(size 1.27 1.27)
+			)
+			(justify left bottom)
 		)
 	)
@@
 		)
 	)
+	(label "GPIO[17..24]"
+		(at 226.06 228.6 90)
+		(effects
+			(font
+				(size 1.27 1.27)
+			)
+			(justify left bottom)
+		)
+	)
+	(label "MCU_SPI2_ADC1"
+		(at 208.28 147.32 90)
+		(effects
+			(font
+				(size 1.27 1.27)
+			)
+			(justify left bottom)
+		)
+	)
 	(label "RMII{RMII}"
 		(at 213.36 73.66 90)
@@
 		)
 	)
+	(label "MCU_SPI6_ADC4"
+		(at 215.9 147.2053 90)
+		(effects
+			(font
+				(size 1.27 1.27)
+			)
+			(justify left bottom)
+		)
+	)
+	(label "GPIO[9..16]"
+		(at 198.12 228.6 90)
+		(effects
+			(font
+				(size 1.27 1.27)
+			)
+			(justify left bottom)
+		)
+	)
 	(label "SDMMC{MMC}"
 		(at 240.03 102.87 0)
@@
 	(label "MDI{MDI}"
 		(at 189.23 31.75 0)
+		(effects
+			(font
+				(size 1.27 1.27)
+			)
+			(justify left bottom)
+		)
+	)
+	(label "GPIO[1..8]"
+		(at 170.18 228.6 90)
+		(effects
+			(font
+				(size 1.27 1.27)
+			)
+			(justify left bottom)
+		)
+	)
+	(label "MCU_SPI5_ADC3"
+		(at 213.36 147.32 90)
+		(effects
+			(font
+				(size 1.27 1.27)
+			)
+			(justify left bottom)
+		)
+	)
+	(label "MCU_SPI3_ADC2"
+		(at 210.82 147.32 90)
 		(effects
 			(font
@@
 	)
 	(sheet
-		(at 162.56 223.52)
+		(at 104.14 212.09)
 		(size 15.24 26.67)
 		(exclude_from_sim no)
@@
 		)
 		(property "Sheetname" "ADC Filter"
-			(at 162.56 222.8084 0)
+			(at 104.14 211.3784 0)
 			(effects
 				(font
@@
 		)
 		(property "Sheetfile" "adc_filt.kicad_sch"
-			(at 162.56 250.7746 0)
+			(at 104.14 239.3446 0)
 			(effects
 				(font
@@
 		(on_board yes)
 		(dnp no)
-		(fields_autoplaced yes)
 		(stroke
 			(width 0.1524)
@@
 		)
 		(property "Sheetname" "DAQ Connector"
-			(at 195.58 241.8584 0)
+			(at 195.58 270.256 0)
 			(effects
 				(font
@@
 		)
 		(property "Sheetfile" "daq_conn.kicad_sch"
-			(at 195.58 268.5546 0)
+			(at 195.58 271.526 0)
 			(effects
 				(font
@@
 			)
 		)
+		(pin "ADC[1..8]" bidirectional
+			(at 204.47 242.57 90)
+			(effects
+				(font
+					(size 1.27 1.27)
+				)
+				(justify right)
+			)
+		)
+		(pin "ADC[9..16]" bidirectional
+			(at 208.28 242.57 90)
+			(effects
+				(font
+					(size 1.27 1.27)
+				)
+				(justify right)
+			)
+		)
+		(pin "ADC[17..24]" bidirectional
+			(at 212.09 242.57 90)
+			(effects
+				(font
+					(size 1.27 1.27)
+				)
+				(justify right)
+			)
+		)
+		(pin "ADC[24..32]" bidirectional
+			(at 215.9 242.57 90)
+			(effects
+				(font
+					(size 1.27 1.27)
+				)
+				(justify right)
+			)
+		)

Commit message: did stuff
Other:
- sheet DAQ Connector ports: added ADC[25..32]; removed ADC[24..32]
- sheet MCU ports: added USB{USB}; removed USB_FS{USB}, USB_HS{USB}
