File: eth_conn.kicad_sch (KiCad schematic)
At the start: 23 parts, among them J1 RJ45

Commit message: did stuff
Parts:
- J1: footprint (none) -> Connector_RJ:RJ45_Amphenol_54602-x08_Horizontal
Connections:
- net SHIELD renamed ETH_SHIELD
Other:
- moved on the sheet: C35, R36

Commit message: did stuff
Parts:
- added U5, U6: ~, CDHD01:CDHD01, symbol CDHD01:CDHD01
Other:
- moved on the sheet: J1, R31, R32, R33, R34, TP23, TP25, TP84, TP85, TP86, TP87, TP88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

Commit message: stuff
Other:
- note added: "Ethernet Connector"
- note removed: "Ethernet PHY"
Changed lines of the file:
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@@
 		)
 	)
-	(text "Ethernet PHY"
+	(text "Ethernet Connector"
 		(exclude_from_sim no)
 		(at 200.406 43.688 0)

Commit message: did 3v3 reg
Parts:
- C36, C37: footprint (none) -> Capacitor_SMD:C_0402_1005Metric
- R29, R30, R31, R32, R33, R34: footprint (none) -> Resistor_SMD:R_0402_1005Metric
Changed lines of the file:
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@@
 			)
 		)
-		(property "Footprint" ""
+		(property "Footprint" "Resistor_SMD:R_0402_1005Metric"
 			(at 203.962 158.75 90)
 			(effects
@@
 			)
 		)
-		(property "Footprint" ""
+		(property "Footprint" "Capacitor_SMD:C_0402_1005Metric"
 			(at 169.8752 160.02 0)
 			(effects
@@
 			)
 		)
-		(property "Footprint" ""
+		(property "Footprint" "Resistor_SMD:R_0402_1005Metric"
 			(at 279.4 140.208 90)
 			(effects
@@
 			)
 		)
-		(property "Footprint" ""
+		(property "Footprint" "Resistor_SMD:R_0402_1005Metric"
 			(at 279.4 144.272 90)
 			(effects
@@
 			)
 		)
-		(property "Footprint" ""
+		(property "Footprint" "Capacitor_SMD:C_0402_1005Metric"
 			(at 155.9052 160.02 0)
 			(effects
@@
 			)
 		)
-		(property "Footprint" ""
+		(property "Footprint" "Resistor_SMD:R_0402_1005Metric"
 			(at 276.352 158.75 90)
 			(effects
@@
 			)
 		)
-		(property "Footprint" ""
+		(property "Footprint" "Resistor_SMD:R_0402_1005Metric"
 			(at 214.122 158.75 90)
 			(effects
@@
 			)
 		)
-		(property "Footprint" ""
+		(property "Footprint" "Resistor_SMD:R_0402_1005Metric"
 			(at 267.462 158.75 90)
 			(effects

Commit message: stuff
Parts:
- added R1, R53, R54, R55: 0, Resistor_SMD:R_0402_1005Metric, symbol Device:R
Connections:
- net MX3-: now also R54.2
- net MX4-: now also R55.2
- net CTREF2: now reaches R29.1, TR1.15 (C_TX)
- net CTREF2: now also R53.1
- net POE_V+: now reaches U6.1 (+)
- net POE_V+: now also U5.1 (+)
- net POE_V-: now reaches U6.2 (-)
- net POE_V-: now also U5.2 (-)
- net POE_CT2: now reaches U6.3
- net POE_CT2: now also R53.2
- net POE_CT1: now reaches U6.4
- net POE_CT1: now also R1.2
- net at U5.3: now also R55.1
- net at U5.4: now also R54.1
- net CTREF1: now reaches R30.1, TR1.10 (C_RX)
- net CTREF1: now also R1.1
Other:
- note added: "CAD Note: Inside dotted line is solid plane connected to SHIELD 2kV isolation to nets outside area PoE circuits are also inside the area"
- note added: "DNM"
- note removed: "CAD Note: Inside dotted line is solid plane connected to SHIELD 2kV isolation to nets outside area"
- moved on the sheet: C33, R31, R32, U5, U6

Commit message: did stuff
Parts:
- renumbered C34 to C33, C36 to C34, C37 to C35, C33 to C36, C35 to C37, R35 to R32, R54 to R33, R55 to R34, R1 to R35, R33 to R36, R53 to R37, R34 to R38, R29 to R39, R30 to R40, R31 to R41, R32 to R42, R36 to R43, TP89 to TP82, TP23 to TP83, TP25 to TP84, TP84 to TP85, TP85 to TP86, TP86 to TP87, TP87 to TP88, TP88 to TP89, U5 to U3, U6 to U4

Commit message: did some layouting
Parts:
- U3, U4: value ~ -> (none)

Commit message: lots
Parts:
- added D39: SMBJ58A, Diode_SMD:D_SMB, symbol Device:D_Zener
Connections:
- net POE_V+: now also D39.1 (K)
- net POE_V-: now also D39.2 (A)
Changed lines of the file:
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@@
+	)
+	(junction
+		(at 234.95 115.57)
+		(diameter 0)
+		(color 0 0 0 0)
 	)
 	(junction
@@
 	)
 	(junction
+		(at 229.87 115.57)
+		(diameter 0)
+		(color 0 0 0 0)
+	)
+	(junction
 		(at 265.43 163.83)
 		(diameter 0)
@@
 	)
 	(junction
-		(at 234.95 115.57)
-		(diameter 0)
-		(color 0 0 0 0)
-	)
-	(junction
 		(at 215.9 134.62)
 		(diameter 0)
@@
 		(color 0 0 0 0)
 	)
+	(junction
+		(at 229.87 104.14)
+		(diameter 0)
+		(color 0 0 0 0)
+	)
 	(bus_entry
 		(at 96.52 129.54)
@@
 	(wire
 		(pts
+			(xy 217.17 104.14) (xy 229.87 104.14)
+		)
+		(stroke
+			(width 0)
+			(type default)
+		)
+	)
+	(wire
+		(pts
 			(xy 298.45 130.81) (xy 330.2 130.81)
 		)
@@
 	(wire
 		(pts
-			(xy 223.52 104.14) (xy 252.73 104.14)
-		)
-		(stroke
-			(width 0)
-			(type default)
-		)
-	)
-	(wire
-		(pts
 			(xy 168.91 144.78) (xy 182.88 144.78)
 		)
@@
 	(wire
 		(pts
+			(xy 229.87 115.57) (xy 234.95 115.57)
+		)
+		(stroke
+			(width 0)
+			(type default)
+		)
+	)
+	(wire
+		(pts
 			(xy 175.26 187.96) (xy 175.26 191.77)
 		)
@@
 	(wire
 		(pts
-			(xy 223.52 115.57) (xy 234.95 115.57)
+			(xy 217.17 115.57) (xy 229.87 115.57)
 		)
 		(stroke
@@
 	(wire
 		(pts
+			(xy 229.87 104.14) (xy 229.87 105.41)
+		)
+		(stroke
+			(width 0)
+			(type default)
+		)
+	)
+	(wire
+		(pts
 			(xy 274.32 146.05) (xy 274.32 148.59)
 		)
@@
 	(wire
 		(pts
+			(xy 229.87 104.14) (xy 252.73 104.14)
+		)
+		(stroke
+			(width 0)
+			(type default)
+		)
+	)
+	(wire
+		(pts
 			(xy 233.68 130.81) (xy 243.84 130.81)
 		)
@@
 		(pts
 			(xy 205.74 144.78) (xy 224.79 144.78)
+		)
+		(stroke
+			(width 0)
+			(type default)
+		)
+	)
+	(wire
+		(pts
+			(xy 229.87 113.03) (xy 229.87 115.57)
 		)
 		(stroke
@@
 	)
 	(label "POE_V-"
-		(at 223.52 115.57 0)
+		(at 217.17 115.57 0)
 		(effects
 			(font
@@
 	)
 	(label "POE_V+"
-		(at 223.52 104.14 0)
+		(at 217.17 104.14 0)
 		(effects
 			(font
@@
 	(hierarchical_label "POE_V+"
 		(shape output)
-		(at 223.52 104.14 180)
+		(at 217.17 104.14 180)
 		(effects
 			(font
@@
 	(hierarchical_label "POE_V-"
 		(shape output)
-		(at 223.52 115.57 180)
+		(at 217.17 115.57 180)
 		(effects
 			(font
@@
 					(unit 1)
 				)
+			)
+		)
+	)
+	(symbol
+		(lib_id "Device:D_Zener")
+		(at 229.87 109.22 270)
+		(unit 1)
+		(body_style 1)
+		(exclude_from_sim no)
+		(in_bom yes)
+		(on_board yes)
+		(in_pos_files yes)
+		(dnp no)
+		(fields_autoplaced yes)
+		(property "Reference" "D39"
+			(at 232.41 107.9499 90)
+			(show_name no)
+			(do_not_autoplace no)
+			(effects
+				(font
+					(size 1.27 1.27)
+				)
+				(justify left)
+			)
+		)
+		(property "Value" "SMBJ58A"
+			(at 232.41 110.4899 90)
+			(show_name no)
+			(do_not_autoplace no)
+			(effects
+				(font
+					(size 1.27 1.27)
+				)
+				(justify left)
+			)
+		)
+		(property "Footprint" "Diode_SMD:D_SMB"
+			(at 229.87 109.22 0)
+			(hide yes)
+			(show_name no)
+			(do_not_autoplace no)
+			(effects
+				(font
+					(size 1.27 1.27)
+				)
+			)
+		)
+		(property "Datasheet" ""
+			(at 229.87 109.22 0)
+			(hide yes)
+			(show_name no)
+			(do_not_autoplace no)
+			(effects
+				(font
+					(size 1.27 1.27)
+				)
+			)
+		)
+		(property "Description" "Zener diode"
+			(at 229.87 109.22 0)
+			(hide yes)
+			(show_name no)
+			(do_not_autoplace no)
+			(effects
+				(font
+					(size 1.27 1.27)
+				)
+			)
+		)
+		(pin "2"
+		)
+		(pin "1"
+		)
+		(instances
+			(project "netdaq"
+				(path "/2970f661-65ab-4e2b-aeda-d76d1044f2b8/ea65a3d0-a0be-4201-b06b-091231bedc11"
+					(reference "D39")
+					(unit 1)
+				)
