File: netdaq.kicad_pcb (KiCad board)
At the start: 2 copper layers, 127.5 x 83 mm, 128 parts, among them J1 RJ45, J3 Conn_01x06_Pin, J4 Micro_SD_Card_Det2, U1 PIC32CK1025GC01100-I/4SB, U10 TLA2518IRTER, U11 TLA2518IRTER, U2 LAN8720A-CP, U3 MP6004GQ-P, U4 PD70100ILD-TR, U7 TPS62A01PDDCR, U8 TLA2518IRTER, U9 TLA2518IRTER

Commit message: did stuff
Parts:
- added C100: C, Capacitor_SMD:C_0402_1005Metric, F.Cu at (196.3, 168.4)
- added C101: C, Capacitor_SMD:C_0402_1005Metric, F.Cu at (196.3, 170.4)
- added C38: C, Capacitor_SMD:C_0402_1005Metric, F.Cu at (137.2, 131.2)
- added C39: C, Capacitor_SMD:C_0402_1005Metric, F.Cu at (137.8, 137.8)
- added C40: C, Capacitor_SMD:C_0402_1005Metric, F.Cu at (139.5, 137.8)
- added C41: C, Capacitor_SMD:C_0402_1005Metric, F.Cu at (139.0, 131.2)
- added C42: C, Capacitor_SMD:C_0402_1005Metric, F.Cu at (140.8, 131.2)
- added C43: C, Capacitor_SMD:C_0402_1005Metric, F.Cu at (141.2, 137.8)
- added C44: C, Capacitor_SMD:C_0402_1005Metric, F.Cu at (143.0, 137.8)
- added C45: C, Capacitor_SMD:C_0402_1005Metric, F.Cu at (142.5, 131.2)
- added C46: C, Capacitor_SMD:C_0402_1005Metric, F.Cu at (144.2, 131.2)
- added C47: C, Capacitor_SMD:C_0402_1005Metric, F.Cu at (144.8, 137.8)
- added C48: C, Capacitor_SMD:C_0402_1005Metric, F.Cu at (146.5, 137.8)
- added C49: C, Capacitor_SMD:C_0402_1005Metric, F.Cu at (146.0, 131.2)
- added C50: C, Capacitor_SMD:C_0402_1005Metric, F.Cu at (147.8, 131.2)
- added C51: C, Capacitor_SMD:C_0402_1005Metric, F.Cu at (148.2, 137.8)
- added C52: C, Capacitor_SMD:C_0402_1005Metric, F.Cu at (150.0, 137.8)
- added C53: C, Capacitor_SMD:C_0402_1005Metric, F.Cu at (149.5, 131.2)
- added C54: C, Capacitor_SMD:C_0402_1005Metric, F.Cu at (151.2, 131.2)
- added C55: C, Capacitor_SMD:C_0402_1005Metric, F.Cu at (151.8, 137.8)
- added C56: C, Capacitor_SMD:C_0402_1005Metric, F.Cu at (153.5, 137.8)
- added C57: C, Capacitor_SMD:C_0402_1005Metric, F.Cu at (153.0, 131.2)
- added C58: C, Capacitor_SMD:C_0402_1005Metric, F.Cu at (154.8, 131.2)
- added C59: C, Capacitor_SMD:C_0402_1005Metric, F.Cu at (155.2, 137.8)
- added C60: C, Capacitor_SMD:C_0402_1005Metric, F.Cu at (157.0, 137.8)
- added C61: C, Capacitor_SMD:C_0402_1005Metric, F.Cu at (156.2, 131.2)
- added C62: C, Capacitor_SMD:C_0402_1005Metric, F.Cu at (158.2, 131.2)
- added C63: C, Capacitor_SMD:C_0402_1005Metric, F.Cu at (158.8, 137.8)
- added C64: C, Capacitor_SMD:C_0402_1005Metric, F.Cu at (160.5, 137.8)
- added C65: C, Capacitor_SMD:C_0402_1005Metric, F.Cu at (160.0, 131.2)
- added C66: C, Capacitor_SMD:C_0402_1005Metric, F.Cu at (164.0, 153.5)
- added C67: C, Capacitor_SMD:C_0402_1005Metric, F.Cu at (187.7, 168.4)
- added C68: C, Capacitor_SMD:C_0402_1005Metric, F.Cu at (187.7, 170.4)
- added C69: C, Capacitor_SMD:C_0402_1005Metric, F.Cu at (187.7, 172.4)
- added C70: C, Capacitor_SMD:C_0402_1005Metric, F.Cu at (187.7, 174.4)
- added C71: C, Capacitor_SMD:C_0402_1005Metric, F.Cu at (190.6, 154.7)
- added C72: C, Capacitor_SMD:C_0402_1005Metric, F.Cu at (190.6, 156.6)
- added C73: C, Capacitor_SMD:C_0402_1005Metric, F.Cu at (190.6, 158.6)
- added C74: C, Capacitor_SMD:C_0402_1005Metric, F.Cu at (190.6, 160.6)
- added C75: C, Capacitor_SMD:C_0402_1005Metric, F.Cu at (190.6, 162.5)
- added C76: C, Capacitor_SMD:C_0402_1005Metric, F.Cu at (190.6, 164.5)
- added C77: C, Capacitor_SMD:C_0402_1005Metric, F.Cu at (190.6, 166.5)
- added C78: C, Capacitor_SMD:C_0402_1005Metric, F.Cu at (190.6, 168.4)
- added C79: C, Capacitor_SMD:C_0402_1005Metric, F.Cu at (190.6, 170.4)
- added C80: C, Capacitor_SMD:C_0402_1005Metric, F.Cu at (190.6, 172.4)
- added C81: C, Capacitor_SMD:C_0402_1005Metric, F.Cu at (190.6, 174.4)
- added C82: C, Capacitor_SMD:C_0402_1005Metric, F.Cu at (193.4, 154.7)
- added C83: C, Capacitor_SMD:C_0402_1005Metric, F.Cu at (193.4, 156.6)
- added C84: C, Capacitor_SMD:C_0402_1005Metric, F.Cu at (193.4, 158.6)
- added C85: C, Capacitor_SMD:C_0402_1005Metric, F.Cu at (193.4, 160.6)
- added C86: C, Capacitor_SMD:C_0402_1005Metric, F.Cu at (193.4, 162.5)
- added C87: C, Capacitor_SMD:C_0402_1005Metric, F.Cu at (193.4, 164.5)
- added C88: C, Capacitor_SMD:C_0402_1005Metric, F.Cu at (193.4, 166.5)
- added C89: C, Capacitor_SMD:C_0402_1005Metric, F.Cu at (193.4, 168.4)
- added C90: C, Capacitor_SMD:C_0402_1005Metric, F.Cu at (193.4, 170.4)
- added C91: C, Capacitor_SMD:C_0402_1005Metric, F.Cu at (193.4, 172.4)
- added C92: C, Capacitor_SMD:C_0402_1005Metric, F.Cu at (193.4, 174.4)
- added C93: C, Capacitor_SMD:C_0402_1005Metric, F.Cu at (196.3, 154.7)
- added C94: C, Capacitor_SMD:C_0402_1005Metric, F.Cu at (196.3, 156.6)
- added C95: C, Capacitor_SMD:C_0402_1005Metric, F.Cu at (196.3, 158.6)
- added C96: C, Capacitor_SMD:C_0402_1005Metric, F.Cu at (196.3, 160.6)
- added C97: C, Capacitor_SMD:C_0402_1005Metric, F.Cu at (196.3, 162.5)
- added C98: C, Capacitor_SMD:C_0402_1005Metric, F.Cu at (196.3, 164.5)
- added C99: C, Capacitor_SMD:C_0402_1005Metric, F.Cu at (196.3, 166.5)
- added D10: D_TVS, Diode_SMD:D_SOD-923, F.Cu at (146.8, 136.2)
- added D11: D_TVS, Diode_SMD:D_SOD-923, F.Cu at (148.5, 136.2)
- added D12: D_TVS, Diode_SMD:D_SOD-923, F.Cu at (150.2, 136.2)
- added D13: D_TVS, Diode_SMD:D_SOD-923, F.Cu at (152.0, 136.2)
- added D14: D_TVS, Diode_SMD:D_SOD-923, F.Cu at (153.8, 136.2)
- added D15: D_TVS, Diode_SMD:D_SOD-923, F.Cu at (155.5, 136.2)
- added D16: D_TVS, Diode_SMD:D_SOD-923, F.Cu at (157.2, 136.2)
- added D17: D_TVS, Diode_SMD:D_SOD-923, F.Cu at (159.0, 136.2)
- added D18: D_TVS, Diode_SMD:D_SOD-923, F.Cu at (160.8, 136.2)
- added D19: D_TVS, Diode_SMD:D_SOD-923, F.Cu at (162.5, 136.2)
- added D20: D_TVS, Diode_SMD:D_SOD-923, F.Cu at (164.2, 136.2)
- added D21: D_TVS, Diode_SMD:D_SOD-923, F.Cu at (166.0, 136.2)
- added D22: D_TVS, Diode_SMD:D_SOD-923, F.Cu at (167.8, 136.2)
- added D23: D_TVS, Diode_SMD:D_SOD-923, F.Cu at (169.5, 136.2)
- added D24: D_TVS, Diode_SMD:D_SOD-923, F.Cu at (171.2, 136.2)
- added D25: D_TVS, Diode_SMD:D_SOD-923, F.Cu at (173.0, 136.2)
- added D26: D_TVS, Diode_SMD:D_SOD-923, F.Cu at (174.8, 136.2)
- added D27: D_TVS, Diode_SMD:D_SOD-923, F.Cu at (176.5, 136.2)
- added D28: D_TVS, Diode_SMD:D_SOD-923, F.Cu at (178.2, 136.2)
- added D29: D_TVS, Diode_SMD:D_SOD-923, F.Cu at (180.0, 136.2)
- added D30: D_TVS, Diode_SMD:D_SOD-923, F.Cu at (181.8, 136.2)
- added D31: D_TVS, Diode_SMD:D_SOD-923, F.Cu at (183.5, 136.2)
- added D32: D_TVS, Diode_SMD:D_SOD-923, F.Cu at (185.2, 136.2)
- added D33: D_TVS, Diode_SMD:D_SOD-923, F.Cu at (187.0, 136.2)
- added D34: D_TVS, Diode_SMD:D_SOD-923, F.Cu at (188.8, 136.2)
- added D35: D_TVS, Diode_SMD:D_SOD-923, F.Cu at (190.5, 136.2)
- added D36: D_TVS, Diode_SMD:D_SOD-923, F.Cu at (192.2, 136.2)
- added D47: BAS40-04, Package_TO_SOT_SMD:SOT-23, F.Cu at (148.0, 127.5)
- added D48: BAS40-04, Package_TO_SOT_SMD:SOT-23, F.Cu at (144.5, 127.5)
- added D49: BAS40-04, Package_TO_SOT_SMD:SOT-23, F.Cu at (129.7, 190.2)
- added D5: D_TVS, Diode_SMD:D_SOD-923, F.Cu at (138.0, 136.2)
- added D50: BAS40-04, Package_TO_SOT_SMD:SOT-23, F.Cu at (137.0, 127.5)
- added D51: BAS40-04, Package_TO_SOT_SMD:SOT-23, F.Cu at (134.6, 190.2)
- added D52: BAS40-04, Package_TO_SOT_SMD:SOT-23, F.Cu at (134.6, 194.6)
- added D53: BAS40-04, Package_TO_SOT_SMD:SOT-23, F.Cu at (139.5, 190.2)
- added D54: BAS40-04, Package_TO_SOT_SMD:SOT-23, F.Cu at (139.5, 194.6)
- added D55: BAS40-04, Package_TO_SOT_SMD:SOT-23, F.Cu at (125.0, 167.7)
- added D56: BAS40-04, Package_TO_SOT_SMD:SOT-23, F.Cu at (124.8, 172.8)
- added D57: BAS40-04, Package_TO_SOT_SMD:SOT-23, F.Cu at (129.7, 168.3)
- added D58: BAS40-04, Package_TO_SOT_SMD:SOT-23, F.Cu at (129.7, 172.8)
- added D59: BAS40-04, Package_TO_SOT_SMD:SOT-23, F.Cu at (134.6, 168.3)
- added D6: D_TVS, Diode_SMD:D_SOD-923, F.Cu at (139.8, 136.2)
- added D60: BAS40-04, Package_TO_SOT_SMD:SOT-23, F.Cu at (134.6, 172.8)
- added D61: BAS40-04, Package_TO_SOT_SMD:SOT-23, F.Cu at (139.5, 168.3)
- added D62: BAS40-04, Package_TO_SOT_SMD:SOT-23, F.Cu at (139.5, 172.8)
- added D63: BAS40-04, Package_TO_SOT_SMD:SOT-23, F.Cu at (124.8, 179.2)
- added D64: BAS40-04, Package_TO_SOT_SMD:SOT-23, F.Cu at (124.8, 183.7)
- added D65: BAS40-04, Package_TO_SOT_SMD:SOT-23, F.Cu at (129.7, 179.2)
- added D66: BAS40-04, Package_TO_SOT_SMD:SOT-23, F.Cu at (129.7, 183.7)
- added D67: BAS40-04, Package_TO_SOT_SMD:SOT-23, F.Cu at (134.6, 179.2)
- added D68: BAS40-04, Package_TO_SOT_SMD:SOT-23, F.Cu at (134.6, 183.7)
- added D69: BAS40-04, Package_TO_SOT_SMD:SOT-23, F.Cu at (139.5, 179.2)
- added D7: D_TVS, Diode_SMD:D_SOD-923, F.Cu at (141.5, 136.2)
- added D70: BAS40-04, Package_TO_SOT_SMD:SOT-23, F.Cu at (139.5, 183.7)
- added D71: BAS40-04, Package_TO_SOT_SMD:SOT-23, F.Cu at (124.8, 201.1)
- added D72: BAS40-04, Package_TO_SOT_SMD:SOT-23, F.Cu at (124.8, 205.5)
- added D73: BAS40-04, Package_TO_SOT_SMD:SOT-23, F.Cu at (129.7, 201.1)
- added D74: BAS40-04, Package_TO_SOT_SMD:SOT-23, F.Cu at (129.7, 205.5)
- added D75: BAS40-04, Package_TO_SOT_SMD:SOT-23, F.Cu at (134.6, 201.1)
- added D76: BAS40-04, Package_TO_SOT_SMD:SOT-23, F.Cu at (134.6, 205.5)
- added D77: BAS40-04, Package_TO_SOT_SMD:SOT-23, F.Cu at (139.5, 201.1)
- added D78: BAS40-04, Package_TO_SOT_SMD:SOT-23, F.Cu at (139.5, 205.5)
- added D8: D_TVS, Diode_SMD:D_SOD-923, F.Cu at (143.2, 136.2)
- added D9: D_TVS, Diode_SMD:D_SOD-923, F.Cu at (145.0, 136.2)
- added R44: R, Resistor_SMD:R_0603_1608Metric, F.Cu at (138.0, 134.0)
- added R45: R, Resistor_SMD:R_0603_1608Metric, F.Cu at (139.8, 134.0)
- added R46: R, Resistor_SMD:R_0603_1608Metric, F.Cu at (141.5, 134.0)
- added R47: R, Resistor_SMD:R_0603_1608Metric, F.Cu at (143.2, 134.0)
- added R48: R, Resistor_SMD:R_0603_1608Metric, F.Cu at (145.0, 134.0)
- added R49: R, Resistor_SMD:R_0603_1608Metric, F.Cu at (146.8, 134.0)
- added R50: R, Resistor_SMD:R_0603_1608Metric, F.Cu at (148.5, 134.0)
- added R51: R, Resistor_SMD:R_0603_1608Metric, F.Cu at (150.2, 134.0)
- added R52: R, Resistor_SMD:R_0603_1608Metric, F.Cu at (152.0, 134.0)
- added R53: R, Resistor_SMD:R_0603_1608Metric, F.Cu at (153.8, 134.0)
- added R54: R, Resistor_SMD:R_0603_1608Metric, F.Cu at (155.5, 134.0)
- added R55: R, Resistor_SMD:R_0603_1608Metric, F.Cu at (157.2, 134.0)
- added R56: R, Resistor_SMD:R_0603_1608Metric, F.Cu at (159.0, 134.0)
- added R57: R, Resistor_SMD:R_0603_1608Metric, F.Cu at (160.8, 134.0)
- added R58: R, Resistor_SMD:R_0603_1608Metric, F.Cu at (216.5, 133.5)
- added R59: R, Resistor_SMD:R_0603_1608Metric, F.Cu at (216.5, 136.0)
- added R60: R, Resistor_SMD:R_0603_1608Metric, F.Cu at (216.5, 138.5)
- added R61: R, Resistor_SMD:R_0603_1608Metric, F.Cu at (216.5, 141.0)
- added R62: R, Resistor_SMD:R_0603_1608Metric, F.Cu at (220.5, 120.9)
- added R63: R, Resistor_SMD:R_0603_1608Metric, F.Cu at (220.5, 123.4)
- added R64: R, Resistor_SMD:R_0603_1608Metric, F.Cu at (220.5, 125.9)
- added R65: R, Resistor_SMD:R_0603_1608Metric, F.Cu at (220.5, 128.4)
- added R66: R, Resistor_SMD:R_0603_1608Metric, F.Cu at (220.5, 131.0)
- added R67: R, Resistor_SMD:R_0603_1608Metric, F.Cu at (220.5, 133.5)
- added R68: R, Resistor_SMD:R_0603_1608Metric, F.Cu at (220.5, 136.0)
- added R69: R, Resistor_SMD:R_0603_1608Metric, F.Cu at (220.5, 138.5)
- added R70: R, Resistor_SMD:R_0603_1608Metric, F.Cu at (220.5, 141.0)
- added R71: R, Resistor_SMD:R_0603_1608Metric, F.Cu at (224.5, 120.9)
- added R72: R, Resistor_SMD:R_0603_1608Metric, F.Cu at (224.5, 123.4)
- added R73: R, Resistor_SMD:R_0603_1608Metric, F.Cu at (224.5, 125.9)
- added R74: R, Resistor_SMD:R_0603_1608Metric, F.Cu at (224.5, 128.4)
- added R75: R, Resistor_SMD:R_0603_1608Metric, F.Cu at (224.5, 131.0)
- moved U9 8.50 mm to (79.5, 175.8)
- renumbered C15 to C1, C5 to C10, C48 to C109, C4 to C11, C44 to C110, C46 to C111, C47 to C112, C50 to C113, C49 to C114, C53 to C115, C51 to C116, C52 to C117, C56 to C118, C54 to C119, C3 to C12, C55 to C120, C59 to C121, C57 to C122, C58 to C123, C62 to C124, C60 to C125, C61 to C126, C2 to C13, C1 to C14, C13 to C15, C12 to C16, C11 to C17, C10 to C18, C21 to C19, C14 to C2, C19 to C20, C20 to C21, C25 to C23, C23 to C25, C27 to C26, C28 to C27, C26 to C28, C18 to C3, C36 to C34, C37 to C35, C17 to C4, C16 to C5, C9 to C6, C8 to C7, C7 to C8, C6 to C9, R5 to R1, R3 to R10, R4 to R11, R6 to R12, R21 to R13, R28 to R14, R22 to R15, R17 to R16, R16 to R17, R15 to R18, R13 to R19, R24 to R20, R12 to R21, R14 to R22, R18 to R24, R19 to R25, R20 to R26, R10 to R27, R11 to R28, R25 to R29, R56 to R3, R27 to R30, R26 to R31, R54 to R33, R55 to R34, R1 to R35, R33 to R36, R53 to R37, R34 to R38, R29 to R39, R57 to R4, R30 to R40, R31 to R41, R32 to R42, R58 to R5, R59 to R6, R9 to R7, R7 to R8, R41 to R80, R43 to R81, R44 to R82, R42 to R83, R52 to R84, R51 to R85, R50 to R86, R49 to R87, R48 to R88, R47 to R89, R8 to R9, R46 to R90, R45 to R91, U5 to U3, U6 to U4, U3 to U5, U4 to U6
Connections:
- J2 pad 1: unconnected-(J2-Pin_1-Pad1) -> /DAQ Connector/EXT_ADC1
- J2 pad 10: unconnected-(J2-Pin_10-Pad10) -> /DAQ Connector/EXT_ADC10
- J2 pad 11: unconnected-(J2-Pin_11-Pad11) -> /DAQ Connector/EXT_ADC11
- J2 pad 12: unconnected-(J2-Pin_12-Pad12) -> /DAQ Connector/EXT_ADC12
- J2 pad 13: unconnected-(J2-Pin_13-Pad13) -> /DAQ Connector/EXT_ADC13
- J2 pad 14: unconnected-(J2-Pin_14-Pad14) -> /DAQ Connector/EXT_ADC14
- J2 pad 15: unconnected-(J2-Pin_15-Pad15) -> /DAQ Connector/EXT_ADC15
- J2 pad 16: unconnected-(J2-Pin_16-Pad16) -> /DAQ Connector/EXT_ADC16
- J2 pad 17: unconnected-(J2-Pin_17-Pad17) -> /DAQ Connector/EXT_ADC17
- J2 pad 18: unconnected-(J2-Pin_18-Pad18) -> /DAQ Connector/EXT_ADC18
- J2 pad 19: unconnected-(J2-Pin_19-Pad19) -> /DAQ Connector/EXT_ADC19
- J2 pad 2: unconnected-(J2-Pin_2-Pad2) -> /DAQ Connector/EXT_ADC2
- J2 pad 20: unconnected-(J2-Pin_20-Pad20) -> /DAQ Connector/EXT_ADC20
- J2 pad 21: unconnected-(J2-Pin_21-Pad21) -> /DAQ Connector/EXT_ADC21
- J2 pad 22: unconnected-(J2-Pin_22-Pad22) -> /DAQ Connector/EXT_ADC22
- J2 pad 23: unconnected-(J2-Pin_23-Pad23) -> /DAQ Connector/EXT_ADC23
- J2 pad 24: unconnected-(J2-Pin_24-Pad24) -> /DAQ Connector/EXT_ADC24
- J2 pad 25: unconnected-(J2-Pin_25-Pad25) -> /DAQ Connector/EXT_ADC25
- J2 pad 26: unconnected-(J2-Pin_26-Pad26) -> /DAQ Connector/EXT_ADC26
- J2 pad 27: unconnected-(J2-Pin_27-Pad27) -> /DAQ Connector/EXT_ADC27
- J2 pad 28: unconnected-(J2-Pin_28-Pad28) -> /DAQ Connector/EXT_ADC28
- J2 pad 29: unconnected-(J2-Pin_29-Pad29) -> /DAQ Connector/EXT_ADC29
- J2 pad 3: unconnected-(J2-Pin_3-Pad3) -> /DAQ Connector/EXT_ADC3
- J2 pad 30: unconnected-(J2-Pin_30-Pad30) -> /DAQ Connector/EXT_ADC30
- J2 pad 31: unconnected-(J2-Pin_31-Pad31) -> /DAQ Connector/EXT_ADC31
- J2 pad 32: unconnected-(J2-Pin_32-Pad32) -> /DAQ Connector/EXT_ADC32
- J2 pad 4: unconnected-(J2-Pin_4-Pad4) -> /DAQ Connector/EXT_ADC4
- J2 pad 5: unconnected-(J2-Pin_5-Pad5) -> /DAQ Connector/EXT_ADC5
- J2 pad 6: unconnected-(J2-Pin_6-Pad6) -> /DAQ Connector/EXT_ADC6
- J2 pad 7: unconnected-(J2-Pin_7-Pad7) -> /DAQ Connector/EXT_ADC7
- J2 pad 8: unconnected-(J2-Pin_8-Pad8) -> /DAQ Connector/EXT_ADC8
- J2 pad 9: unconnected-(J2-Pin_9-Pad9) -> /DAQ Connector/EXT_ADC9
- U1 pad 10: /ADC3/SPI.SCK -> /MCU/SPI5.SCK
- U1 pad 11: /ADC3/SPI.CS# -> /MCU/SPI5.CS#
- U1 pad 16: /ADC4/SPI.MOSI -> /MCU/SPI6.MOSI
- U1 pad 17: /ADC4/SPI.MISO -> /MCU/SPI6.MISO
- U1 pad 22: /ADC4/SPI.SCK -> /MCU/SPI6.SCK
- U1 pad 23: /ADC4/SPI.CS# -> /MCU/SPI6.CS#
- U1 pad 45: /ADC2/SPI.MOSI -> /MCU/SPI3.MOSI
- U1 pad 46: /ADC2/SPI.MISO -> /MCU/SPI3.MISO
- U1 pad 47: /ADC2/SPI.SCK -> /MCU/SPI3.SCK
- U1 pad 48: /ADC2/SPI.CS# -> /MCU/SPI3.CS#
- U1 pad 64: /ADC1/SPI.MOSI -> /MCU/SPI2.MOSI
- U1 pad 65: /ADC1/SPI.MISO -> /MCU/SPI2.MISO
- U1 pad 66: /ADC1/SPI.SCK -> /MCU/SPI2.SCK
- U1 pad 67: /ADC1/SPI.CS# -> /MCU/SPI2.CS#
- U1 pad 8: /ADC3/SPI.MOSI -> /MCU/SPI5.MOSI
- U1 pad 9: /ADC3/SPI.MISO -> /MCU/SPI5.MISO
- U10 pad 1: /ADC3/GPIO2 -> /GPIO19
- U10 pad 15: /ADC3/GPIO0 -> /GPIO17
- U10 pad 16: /ADC3/GPIO1 -> /GPIO18
- U10 pad 2: /ADC3/GPIO3 -> /GPIO20
- U10 pad 3: /ADC3/GPIO4 -> /GPIO21
- U10 pad 4: /ADC3/GPIO5 -> /GPIO22
- U10 pad 5: /ADC3/GPIO6 -> /GPIO23
- U10 pad 6: /ADC3/GPIO7 -> /GPIO24
- U11 pad 1: /ADC4/GPIO2 -> /GPIO27
- U11 pad 15: /ADC4/GPIO0 -> /GPIO24
- U11 pad 16: /ADC4/GPIO1 -> /GPIO26
- U11 pad 2: /ADC4/GPIO3 -> /GPIO28
- U11 pad 3: /ADC4/GPIO4 -> /GPIO29
- U11 pad 4: /ADC4/GPIO5 -> /GPIO30
- U11 pad 5: /ADC4/GPIO6 -> /GPIO31
- U11 pad 6: /ADC4/GPIO7 -> /GPIO32
- U8 pad 1: /ADC1/GPIO2 -> /GPIO3
- U8 pad 15: /ADC1/GPIO0 -> /GPIO1
- U8 pad 16: /ADC1/GPIO1 -> /GPIO2
- U8 pad 2: /ADC1/GPIO3 -> /GPIO4
- U8 pad 3: /ADC1/GPIO4 -> /GPIO5
- U8 pad 4: /ADC1/GPIO5 -> /GPIO6
- U8 pad 5: /ADC1/GPIO6 -> /GPIO7
- U8 pad 6: /ADC1/GPIO7 -> /GPIO8
- U9 pad 1: /ADC2/GPIO2 -> /GPIO11
- U9 pad 15: /ADC2/GPIO0 -> /GPIO9
- U9 pad 16: /ADC2/GPIO1 -> /GPIO10
- U9 pad 2: /ADC2/GPIO3 -> /GPIO12
- U9 pad 3: /ADC2/GPIO4 -> /GPIO13
- U9 pad 4: /ADC2/GPIO5 -> /GPIO14
- U9 pad 5: /ADC2/GPIO6 -> /GPIO15
- U9 pad 6: /ADC2/GPIO7 -> /GPIO16
Routing:
- net /DAQ Connector/EXT_ADC1: track 0.00 -> 6.14 mm
- net unconnected-(J2-Pin_38-Pad38): track 0.00 -> 3.72 mm
- net unconnected-(J2-Pin_36-Pad36): track 0.00 -> 3.72 mm
- net unconnected-(J2-Pin_34-Pad34): track 0.00 -> 3.72 mm
- net /DAQ Connector/EXT_ADC32: track 0.00 -> 3.72 mm
- net /DAQ Connector/EXT_ADC30: track 0.00 -> 3.72 mm
- net /DAQ Connector/EXT_ADC8: track 0.00 -> 3.47 mm
- net /DAQ Connector/EXT_ADC6: track 0.00 -> 3.47 mm
- net /DAQ Connector/EXT_ADC4: track 0.00 -> 3.47 mm
- net /DAQ Connector/EXT_ADC28: track 0.00 -> 3.47 mm
- net /DAQ Connector/EXT_ADC26: track 0.00 -> 3.47 mm
- net /DAQ Connector/EXT_ADC24: track 0.00 -> 3.47 mm
- net /DAQ Connector/EXT_ADC22: track 0.00 -> 3.47 mm
- net /DAQ Connector/EXT_ADC20: track 0.00 -> 3.47 mm
- net /DAQ Connector/EXT_ADC2: track 0.00 -> 3.47 mm
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
Commit message: did stuff
Parts:
- R1: value 0 -> 10k
- moved C126 117.1 mm to (190.2, 117.8), turned to 0 degrees
- moved C124 116.7 mm to (190.2, 115.2), turned to 0 degrees
- moved C121 113.3 mm to (176.2, 115.2), turned to 0 degrees
- moved C123 113.2 mm to (176.2, 117.8), turned to 0 degrees
- moved C125 111.0 mm to (186.3, 113.8), turned to 90 degrees
- moved U11 110.9 mm to (185.8, 118.2), turned to 90 degrees
- moved C122 107.8 mm to (172.2, 113.8), turned to 90 degrees
- moved U10 106.8 mm to (171.8, 118.2), turned to 90 degrees
- moved D72 100.1 mm to (187.5, 127.5), turned to 90 degrees
- moved D71 98.9 mm to (190.9, 127.6), turned to 90 degrees
- moved D76 97.6 mm to (187.5, 123.5), turned to 90 degrees
- moved U9 97.1 mm to (157.8, 118.2), turned to 90 degrees
- moved C120 96.8 mm to (162.2, 117.8), turned to 0 degrees
- moved C118 96.6 mm to (162.2, 115.2), turned to 0 degrees
- moved D75 95.9 mm to (191.0, 123.5), turned to 90 degrees
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Connections:
- net /MCU/SPI2.CS# renamed /MCU_SPI2_ADC1.CS#
- net /MCU/SPI2.MISO renamed /MCU_SPI2_ADC1.MISO
- net /MCU/SPI2.MOSI renamed /MCU_SPI2_ADC1.MOSI
- net /MCU/SPI2.SCK renamed /MCU_SPI2_ADC1.SCK
- net /MCU/SPI3.CS# renamed /MCU_SPI3_ADC2.CS#
- net /MCU/SPI3.MISO renamed /MCU_SPI3_ADC2.MISO
- net /MCU/SPI3.MOSI renamed /MCU_SPI3_ADC2.MOSI
- net /MCU/SPI3.SCK renamed /MCU_SPI3_ADC2.SCK
- net /MCU/SPI5.CS# renamed /MCU_SPI5_ADC3.CS#
- net /MCU/SPI5.MISO renamed /MCU_SPI5_ADC3.MISO
- net /MCU/SPI5.MOSI renamed /MCU_SPI5_ADC3.MOSI
- net /MCU/SPI5.SCK renamed /MCU_SPI5_ADC3.SCK
- net /MCU/SPI6.CS# renamed /MCU_SPI6_ADC4.CS#
- net /MCU/SPI6.MISO renamed /MCU_SPI6_ADC4.MISO
- net /MCU/SPI6.MOSI renamed /MCU_SPI6_ADC4.MOSI
- net /MCU/SPI6.SCK renamed /MCU_SPI6_ADC4.SCK
- net /MCU/USB.D+ renamed /USB.D+
- net /MCU/USB.D- renamed /USB.D-
- C101 pad 1: /DAQ Connector/ADC32 -> /GPIO32
- C86 pad 1: /GPIO26 -> /GPIO25
- C89 pad 1: /GPIO27 -> /GPIO26
- C90 pad 1: /GPIO28 -> /GPIO27
- C93 pad 1: /GPIO29 -> /GPIO28
- C94 pad 1: /GPIO30 -> /GPIO29
- C97 pad 1: /GPIO31 -> /GPIO30
- C98 pad 1: /GPIO32 -> /GPIO31
- D74 pad 3: /GPIO24 -> /GPIO25
- R1 pad 1: /MCU/PA01 -> +3.3V
- R1 pad 2: /MCU/SPI7.MOSI -> /MCU/RESET#
- R68 pad 1: /GPIO26 -> /GPIO25
- R69 pad 1: /GPIO27 -> /GPIO26
- R70 pad 1: /GPIO28 -> /GPIO27
- R71 pad 1: /GPIO29 -> /GPIO28
- R72 pad 1: /GPIO30 -> /GPIO29
- R73 pad 1: /GPIO31 -> /GPIO30
- R74 pad 1: /GPIO32 -> /GPIO31
- R75 pad 1: /DAQ Connector/ADC32 -> /GPIO32
Routing:
- net /GPIO9: track 0.00 -> 19.2 mm
- net /GPIO10: track 0.00 -> 18.3 mm
- net /GPIO15: track 0.00 -> 17.7 mm
- net /GPIO16: track 0.00 -> 17.6 mm
- net /GPIO12: track 0.00 -> 16.5 mm
- net /GPIO11: track 0.00 -> 16.3 mm
- net /GPIO13: track 0.00 -> 16.0 mm
- net /GPIO14: track 0.00 -> 15.0 mm
- net /GPIO6: track 0.00 -> 13.0 mm
- net /GPIO8: track 0.00 -> 13.0 mm
- net /GPIO4: track 0.00 -> 13.0 mm
- net /GPIO2: track 0.00 -> 13.0 mm
- net /GPIO7: track 0.00 -> 8.58 mm
- net /GPIO17: track 0.00 -> 8.58 mm
- net /GPIO5: track 0.00 -> 8.53 mm
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
Commit message: did stuff
Parts:
- moved TR1 159.4 mm to (170.0, 75.3)
- moved C114 158.9 mm to (105.1, 97.5), turned to -90 degrees
- moved J1 157.8 mm to (174.3, 61.1)
- moved C113 156.6 mm to (107.6, 98.3), turned to -90 degrees
- moved C6 155.7 mm to (184.5, 112.0), turned to 180 degrees
- moved R84 153.1 mm to (110.1, 97.5), turned to -90 degrees
- moved R85 150.7 mm to (112.1, 97.5), turned to -90 degrees
- moved R86 148.4 mm to (114.0, 97.5), turned to -90 degrees
- moved C4 147.1 mm to (186.4, 106.0), turned to 0 degrees
- moved C13 146.5 mm to (180.8, 111.2), turned to 0 degrees
- moved R87 146.2 mm to (116.0, 97.5), turned to -90 degrees
- moved R88 143.9 mm to (118.0, 97.5), turned to -90 degrees
- moved R89 141.7 mm to (120.0, 97.5), turned to -90 degrees
- moved R90 139.5 mm to (122.0, 97.5), turned to -90 degrees
- moved C5 138.4 mm to (183.5, 105.9), turned to 0 degrees
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Connections:
- J2 pad 1: /DAQ Connector/EXT_ADC1 -> unconnected-(J2-Pin_1-Pad1)
- J2 pad 10: /DAQ Connector/EXT_ADC10 -> /DAQ Connector/EXT_ADC6
- J2 pad 11: /DAQ Connector/EXT_ADC11 -> /DAQ Connector/EXT_ADC7
- J2 pad 12: /DAQ Connector/EXT_ADC12 -> /DAQ Connector/EXT_ADC8
- J2 pad 13: /DAQ Connector/EXT_ADC13 -> /DAQ Connector/EXT_ADC9
- J2 pad 14: /DAQ Connector/EXT_ADC14 -> /DAQ Connector/EXT_ADC10
- J2 pad 15: /DAQ Connector/EXT_ADC15 -> /DAQ Connector/EXT_ADC11
- J2 pad 16: /DAQ Connector/EXT_ADC16 -> /DAQ Connector/EXT_ADC12
- J2 pad 17: /DAQ Connector/EXT_ADC17 -> /DAQ Connector/EXT_ADC13
- J2 pad 18: /DAQ Connector/EXT_ADC18 -> /DAQ Connector/EXT_ADC14
- J2 pad 19: /DAQ Connector/EXT_ADC19 -> /DAQ Connector/EXT_ADC15
- J2 pad 2: /DAQ Connector/EXT_ADC2 -> unconnected-(J2-Pin_2-Pad2)
- J2 pad 20: /DAQ Connector/EXT_ADC20 -> /DAQ Connector/EXT_ADC16
- J2 pad 21: /DAQ Connector/EXT_ADC21 -> /DAQ Connector/EXT_ADC17
- J2 pad 22: /DAQ Connector/EXT_ADC22 -> /DAQ Connector/EXT_ADC18
- J2 pad 23: /DAQ Connector/EXT_ADC23 -> /DAQ Connector/EXT_ADC19
- J2 pad 24: /DAQ Connector/EXT_ADC24 -> /DAQ Connector/EXT_ADC20
- J2 pad 25: /DAQ Connector/EXT_ADC25 -> /DAQ Connector/EXT_ADC21
- J2 pad 26: /DAQ Connector/EXT_ADC26 -> /DAQ Connector/EXT_ADC22
- J2 pad 27: /DAQ Connector/EXT_ADC27 -> /DAQ Connector/EXT_ADC23
- J2 pad 28: /DAQ Connector/EXT_ADC28 -> /DAQ Connector/EXT_ADC24
- J2 pad 29: /DAQ Connector/EXT_ADC29 -> /DAQ Connector/EXT_ADC25
- J2 pad 3: /DAQ Connector/EXT_ADC3 -> unconnected-(J2-Pin_3-Pad3)
- J2 pad 30: /DAQ Connector/EXT_ADC30 -> /DAQ Connector/EXT_ADC26
- J2 pad 31: /DAQ Connector/EXT_ADC31 -> /DAQ Connector/EXT_ADC27
- J2 pad 32: /DAQ Connector/EXT_ADC32 -> /DAQ Connector/EXT_ADC28
- J2 pad 33: unconnected-(J2-Pin_33-Pad33) -> /DAQ Connector/EXT_ADC29
- J2 pad 34: unconnected-(J2-Pin_34-Pad34) -> /DAQ Connector/EXT_ADC30
- J2 pad 35: unconnected-(J2-Pin_35-Pad35) -> /DAQ Connector/EXT_ADC31
- J2 pad 36: unconnected-(J2-Pin_36-Pad36) -> /DAQ Connector/EXT_ADC32
- J2 pad 37: unconnected-(J2-Pin_37-Pad37) -> GND
- J2 pad 38: unconnected-(J2-Pin_38-Pad38) -> GND
- J2 pad 4: /DAQ Connector/EXT_ADC4 -> unconnected-(J2-Pin_4-Pad4)
- J2 pad 5: /DAQ Connector/EXT_ADC5 -> /DAQ Connector/EXT_ADC1
- J2 pad 6: /DAQ Connector/EXT_ADC6 -> /DAQ Connector/EXT_ADC2
- J2 pad 7: /DAQ Connector/EXT_ADC7 -> /DAQ Connector/EXT_ADC3
- J2 pad 8: /DAQ Connector/EXT_ADC8 -> /DAQ Connector/EXT_ADC4
- J2 pad 9: /DAQ Connector/EXT_ADC9 -> /DAQ Connector/EXT_ADC5
- U1 pad 10: /MCU_SPI5_ADC3.SCK -> /ADC2/SPI.SCK
- U1 pad 11: /MCU_SPI5_ADC3.CS# -> /ADC2/SPI.CS#
- U1 pad 16: /MCU_SPI6_ADC4.MOSI -> /MCU_SPI5_ADC3.MOSI
- U1 pad 17: /MCU_SPI6_ADC4.MISO -> /MCU_SPI5_ADC3.MISO
- U1 pad 22: /MCU_SPI6_ADC4.SCK -> /MCU_SPI5_ADC3.SCK
- U1 pad 23: /MCU_SPI6_ADC4.CS# -> /MCU_SPI5_ADC3.CS#
- U1 pad 45: /MCU_SPI3_ADC2.MOSI -> /MCU_SPI6_ADC4.MOSI
- U1 pad 46: /MCU_SPI3_ADC2.MISO -> /MCU_SPI6_ADC4.MISO
- U1 pad 47: /MCU_SPI3_ADC2.SCK -> /MCU_SPI6_ADC4.SCK
- U1 pad 48: /MCU_SPI3_ADC2.CS# -> /MCU_SPI6_ADC4.CS#
- U1 pad 8: /MCU_SPI5_ADC3.MOSI -> /ADC2/SPI.MOSI
- U1 pad 9: /MCU_SPI5_ADC3.MISO -> /ADC2/SPI.MISO
- U10 pad 11: /ADC3/SPI.CS# -> /MCU_SPI5_ADC3.CS#
- U10 pad 12: /ADC3/SPI.MISO -> /MCU_SPI5_ADC3.MISO
- U10 pad 13: /ADC3/SPI.SCK -> /MCU_SPI5_ADC3.SCK
- U10 pad 14: /ADC3/SPI.MOSI -> /MCU_SPI5_ADC3.MOSI
- U11 pad 11: /ADC4/SPI.CS# -> /MCU_SPI6_ADC4.CS#
- U11 pad 12: /ADC4/SPI.MISO -> /MCU_SPI6_ADC4.MISO
- U11 pad 13: /ADC4/SPI.SCK -> /MCU_SPI6_ADC4.SCK
- U11 pad 14: /ADC4/SPI.MOSI -> /MCU_SPI6_ADC4.MOSI
- U11 pad 15: /GPIO24 -> /GPIO25
- U8 pad 11: /ADC1/SPI.CS# -> /MCU_SPI2_ADC1.CS#
- U8 pad 12: /ADC1/SPI.MISO -> /MCU_SPI2_ADC1.MISO
- U8 pad 13: /ADC1/SPI.SCK -> /MCU_SPI2_ADC1.SCK
- U8 pad 14: /ADC1/SPI.MOSI -> /MCU_SPI2_ADC1.MOSI
Routing:
- net /ADC2/SPI.MOSI: track 0.00 -> 14.4 mm
- net /ADC2/SPI.SCK: track 0.00 -> 13.3 mm
- net /ADC2/SPI.MISO: track 0.00 -> 12.1 mm, vias 0 -> 2
- net /ADC2/SPI.CS#: track 0.00 -> 11.8 mm
- net /MCU_SPI5_ADC3.MOSI: track 0.00 -> 8.57 mm
- net /MCU_SPI5_ADC3.MISO: track 0.00 -> 8.14 mm, vias 0 -> 2
- net /MCU_SPI5_ADC3.SCK: track 0.00 -> 6.69 mm
- net /MCU_SPI5_ADC3.CS#: track 0.00 -> 6.08 mm
- net unconnected-(J2-Pin_38-Pad38): track 3.72 -> 0.00 mm
- net unconnected-(J2-Pin_36-Pad36): track 3.72 -> 0.00 mm
- net unconnected-(J2-Pin_34-Pad34): track 3.72 -> 0.00 mm
- net GND: track 1.09 -> 4.82 mm
- net unconnected-(J2-Pin_4-Pad4): track 0.00 -> 3.47 mm
- net /DAQ Connector/EXT_ADC2: track 3.86 -> 7.33 mm
- net Net-(U9-DECAP): track 0.00 -> 3.19 mm
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Other:
- board size 127.5 x 83 mm -> 131.5 x 93 mm

Commit message: stuff
Parts:
- moved C35 219.7 mm to (141.5, 79.0), turned to -90 degrees
- moved U5 218.0 mm to (179.0, 58.7)
- moved C34 213.0 mm to (148.0, 79.0), turned to -90 degrees
- moved R34 205.6 mm to (155.5, 55.5), turned to 180 degrees
- moved R33 204.4 mm to (155.5, 61.5), turned to 180 degrees
- moved R37 203.8 mm to (155.5, 64.5)
- moved R35 203.4 mm to (155.5, 66.0)
- moved R38 201.1 mm to (155.5, 54.0)
- moved R36 199.5 mm to (155.5, 58.5), turned to 180 degrees
- moved R42 199.3 mm to (155.5, 57.0)
- moved R41 198.2 mm to (155.5, 60.0)
- moved R39 196.8 mm to (155.5, 63.0)
- moved R40 196.4 mm to (155.5, 67.5)
- moved TR2 192.7 mm to (186.1, 66.0), turned to -90 degrees
- moved U3 187.0 mm to (161.5, 58.0), turned to -90 degrees
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Connections:
- net /ADC2/SPI.CS# renamed /MCU_SPI3_ADC2.CS#
- net /ADC2/SPI.MISO renamed /MCU_SPI3_ADC2.MISO
- net /ADC2/SPI.MOSI renamed /MCU_SPI3_ADC2.MOSI
- net /ADC2/SPI.SCK renamed /MCU_SPI3_ADC2.SCK
- R13 pad 2: /Ethernet PHY/RMII.REFCK -> /RMII.REFCK
- R15 pad 2: /Ethernet PHY/RMII.RXER -> /RMII.RXER
- R19 pad 2: /Ethernet PHY/RMII.RXD0 -> /RMII.RXD0
- R21 pad 2: /Ethernet PHY/RMII.RXD1 -> /RMII.RXD1
- R22 pad 2: /Ethernet PHY/RMII.CRSDV -> /RMII.CRSDV
- R23 pad 1: /Ethernet PHY/RMII.RXER -> /RMII.RXER
- U1 pad 51: /MCU/RMII.REFCK -> /RMII.REFCK
- U1 pad 60: /MCU/RMII.RXD1 -> /RMII.RXD1
- U1 pad 61: /MCU/RMII.RXD0 -> /RMII.RXD0
- U1 pad 63: /MCU/RMII.RXER -> /RMII.RXER
- U1 pad 68: /MCU/RMII.CRSDV -> /RMII.CRSDV
- U1 pad 71: /MCU/RMII.TXEN -> /RMII.TXEN
- U1 pad 72: /MCU/RMII.TXD0 -> /RMII.TXD0
- U1 pad 73: /MCU/RMII.TXD1 -> /RMII.TXD1
- U2 pad 10: /Ethernet PHY/RMII.RXER -> /RMII.RXER
- U2 pad 14: /Ethernet PHY/RMII.REFCK -> /RMII.REFCK
- U2 pad 16: /Ethernet PHY/RMII.TXEN -> /RMII.TXEN
- U2 pad 17: /Ethernet PHY/RMII.TXD0 -> /RMII.TXD0
- U2 pad 18: /Ethernet PHY/RMII.TXD1 -> /RMII.TXD1
Routing:
- net /SDMMC.SDDAT0: track 0.00 -> 30.8 mm
- net /SDMMC.SDDAT2: track 0.00 -> 21.7 mm, vias 0 -> 2
- net /Ethernet Connector/MX4-: track 0.00 -> 20.8 mm
- net /SDMMC.SDDAT3: track 0.00 -> 20.6 mm, vias 0 -> 2
- net /SDMMC.SDCMD: track 0.00 -> 20.5 mm
- net /Ethernet Connector/MX4+: track 0.00 -> 17.6 mm
- net /Ethernet Connector/MX3-: track 0.00 -> 16.6 mm
- net Net-(C36-Pad1): track 0.00 -> 16.1 mm
- net /SDMMC.SDDAT1: track 0.00 -> 16.0 mm
- net /Ethernet Connector/MX3+: track 0.00 -> 12.5 mm
- net /Ethernet Connector/CTREF2: track 0.00 -> 12.2 mm
- net /SDMMC.SDWP: track 0.00 -> 11.3 mm
- net /SDMMC.SDCK: track 0.00 -> 11.3 mm
- net /Ethernet Connector/MX2+: track 0.00 -> 9.68 mm
- net /Ethernet Connector/MX1+: track 0.00 -> 7.20 mm
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
Commit message: did some layouting
Parts:
- added Y4: Crystal_GND24, Crystal:Crystal_SMD_Abracon_ABM8G-4Pin_3.2x2.5mm, F.Cu at (136.8, 89.8)
- moved R1 130.3 mm to (235.6, 111.4)
- moved R10 130.3 mm to (235.6, 107.4)
- moved R11 130.3 mm to (235.6, 109.4)
- moved R12 130.3 mm to (235.6, 113.4)
- moved R7 130.3 mm to (235.6, 119.4)
- moved R8 130.3 mm to (235.6, 115.4)
- moved R9 130.3 mm to (235.6, 117.4)
- moved C19 130.3 mm to (238.5, 117.4)
- moved C20 130.3 mm to (238.5, 113.5)
- moved C21 130.3 mm to (238.5, 115.5)
- moved C22 130.3 mm to (238.5, 119.4)
- moved D1 130.3 mm to (239.3, 108.0)
- moved D2 130.3 mm to (239.3, 111.0)
- moved R1 130.3 mm to (231.5, 115.4)
- moved R2 130.3 mm to (231.5, 117.4)
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Routing:
- net /SMI.MDC: track 2.33 -> 47.8 mm, vias 0 -> 2
- net /SMI.MDIO: track 3.90 -> 47.7 mm, vias 0 -> 2
- net /RMII.RXD1: track 0.00 -> 43.4 mm, vias 0 -> 4
- net /RMII.RXD0: track 0.00 -> 40.8 mm, vias 0 -> 4
- net /RMII.REFCK: track 2.15 -> 38.5 mm, vias 0 -> 2
- net /MCU_SPI2_ADC1.MOSI: track 0.00 -> 36.0 mm, vias 0 -> 2
- net /MCU_SPI2_ADC1.SCK: track 0.00 -> 33.7 mm, vias 0 -> 2
- net /SDMMC.SDCD: track 0.00 -> 33.2 mm
- net /MCU_SPI2_ADC1.MISO: track 0.00 -> 33.0 mm, vias 0 -> 2
- net /MCU_SPI2_ADC1.CS#: track 0.00 -> 32.2 mm, vias 0 -> 2
- net /RMII.RXER: track 2.83 -> 34.3 mm, vias 0 -> 4
- net /RMII.TXD1: track 0.00 -> 27.6 mm, vias 0 -> 2
- net /RMII.TXD0: track 0.00 -> 27.2 mm, vias 0 -> 2
- net /RMII.TXEN: track 0.00 -> 26.9 mm
- net /RMII.CRSDV: track 0.00 -> 26.7 mm, vias 0 -> 2
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