File: daq_conn.kicad_sch (KiCad schematic)
At the start: 161 parts

Commit message: fixed a bunch of errors, set pin type on alot of pins
Parts:
- J2: value (none) -> DMC 1,5/19-G1F-3,5-LR P26THR
Changed lines of the file:
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@@
 			)
 		)
-		(property "Value" ""
+		(property "Value" "DMC 1,5/19-G1F-3,5-LR P26THR"
 			(at 212.09 102.87 0)
 			(show_name no)

Commit message: did some placement/routing of adc input stage
Parts:
- R44, R45, R46, R47, R48, R49, R50, R51, R52, R53, R54, R55, R56, R57, R58, R59, R60, R61, R62, R63, R64, R65, R66, R67, R68, R69, R70, R71, R72, R73, R74, R75: footprint Resistor_SMD:R_1210_3225Metric -> Resistor_SMD:R_0402_1005Metric; LCSC C5576460 -> C11702; LCSC Part C5576460 -> C11702

Commit message: did stuff
Parts:
- C100, C39, C40, C43, C44, C47, C48, C51, C52, C55, C56, C59, C60, C63, C64, C67, C68, C71, C72, C75, C76, C79, C80, C83, C84, C87, C88, C91, C92, C95, C96, C99: LCSC (none) -> C1523; LCSC Basic/Pref (none) -> y; LCSC Part (none) -> C1523
- R44, R45, R46, R47, R48, R49, R50, R51, R52, R53, R54, R55, R56, R57, R58, R59, R60, R61, R62, R63, R64, R65, R66, R67, R68, R69, R70, R71, R72, R73, R74, R75: LCSC Basic/Pref n -> y

Commit message: did stuff
Parts:
- J2: LCSC missing (none) -> y
Connections:
- net GND: now also J2.1 (Pin_1), J2.2 (Pin_2), J2.3 (Pin_3), J2.4 (Pin_4)
Changed lines of the file:
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@@
 	)
 	(junction
+		(at 227.33 107.95)
+		(diameter 0)
+		(color 0 0 0 0)
+	)
+	(junction
+		(at 196.85 107.95)
+		(diameter 0)
+		(color 0 0 0 0)
+	)
+	(junction
 		(at 295.91 208.28)
 		(diameter 0)
@@
 	(wire
 		(pts
+			(xy 196.85 107.95) (xy 198.12 107.95)
+		)
+		(stroke
+			(width 0)
+			(type default)
+		)
+	)
+	(wire
+		(pts
 			(xy 295.91 231.14) (xy 295.91 232.41)
 		)
@@
 	(wire
 		(pts
+			(xy 196.85 102.87) (xy 196.85 107.95)
+		)
+		(stroke
+			(width 0)
+			(type default)
+		)
+	)
+	(wire
+		(pts
 			(xy 295.91 68.58) (xy 295.91 67.31)
 		)
@@
 	(wire
 		(pts
+			(xy 196.85 107.95) (xy 196.85 110.49)
+		)
+		(stroke
+			(width 0)
+			(type default)
+		)
+	)
+	(wire
+		(pts
 			(xy 96.52 109.22) (xy 96.52 110.49)
 		)
@@
 	(wire
 		(pts
+			(xy 196.85 110.49) (xy 198.12 110.49)
+		)
+		(stroke
+			(width 0)
+			(type default)
+		)
+	)
+	(wire
+		(pts
 			(xy 96.52 67.31) (xy 106.68 67.31)
 		)
@@
 	(wire
 		(pts
+			(xy 227.33 107.95) (xy 226.06 107.95)
+		)
+		(stroke
+			(width 0)
+			(type default)
+		)
+	)
+	(wire
+		(pts
 			(xy 295.91 175.26) (xy 295.91 176.53)
 		)
@@
 	(wire
 		(pts
+			(xy 227.33 102.87) (xy 227.33 107.95)
+		)
+		(stroke
+			(width 0)
+			(type default)
+		)
+	)
+	(wire
+		(pts
 			(xy 127 110.49) (xy 127 109.22)
 		)
@@
 	(wire
 		(pts
+			(xy 227.33 107.95) (xy 227.33 110.49)
+		)
+		(stroke
+			(width 0)
+			(type default)
+		)
+	)
+	(wire
+		(pts
 			(xy 226.06 135.89) (xy 264.16 135.89)
 		)
@@
 	(wire
 		(pts
+			(xy 227.33 110.49) (xy 226.06 110.49)
+		)
+		(stroke
+			(width 0)
+			(type default)
+		)
+	)
+	(wire
+		(pts
 			(xy 326.39 81.28) (xy 326.39 82.55)
 		)
@@
 		(in_pos_files yes)
 		(dnp no)
-		(fields_autoplaced yes)
 		(property "Reference" "J2"
-			(at 212.09 100.33 0)
+			(at 212.09 95.504 0)
 			(show_name no)
 			(do_not_autoplace no)
@@
 		)
 		(property "Value" "DMC 1,5/19-G1F-3,5-LR P26THR"
-			(at 212.09 102.87 0)
+			(at 212.09 98.044 0)
 			(show_name no)
 			(do_not_autoplace no)
@@
 			)
 		)
-		(property "LCSC missing" ""
+		(property "LCSC missing" "y"
 			(at 212.09 104.14 0)
 			(hide yes)
@@
 	)
 	(symbol
+		(lib_id "power:GND")
+		(at 227.33 102.87 180)
+		(unit 1)
+		(body_style 1)
+		(exclude_from_sim no)
+		(in_bom yes)
+		(on_board yes)
+		(in_pos_files yes)
+		(dnp no)
+		(property "Reference" "#PWR0552"
+			(at 227.33 96.52 0)
+			(hide yes)
+			(show_name no)
+			(do_not_autoplace no)
+			(effects
+				(font
+					(size 1.27 1.27)
+				)
+			)
+		)
+		(property "Value" "GND"
+			(at 223.266 101.092 0)
+			(show_name no)
+			(do_not_autoplace no)
+			(effects
+				(font
+					(size 1.27 1.27)
+				)
+			)
+		)
+		(property "Footprint" ""
+			(at 227.33 102.87 0)
+			(hide yes)
+			(show_name no)
+			(do_not_autoplace no)
+			(effects
+				(font
+					(size 1.27 1.27)
+				)
+			)
+		)
+		(property "Datasheet" ""
+			(at 227.33 102.87 0)
+			(hide yes)
+			(show_name no)
+			(do_not_autoplace no)
+			(effects
+				(font
+					(size 1.27 1.27)
+				)
+			)
+		)
+		(property "Description" "Power symbol creates a global label with name \"GND\" , ground"
+			(at 227.33 102.87 0)
+			(hide yes)
+			(show_name no)
+			(do_not_autoplace no)
+			(effects
+				(font
+					(size 1.27 1.27)
+				)
+			)
+		)
+		(pin "1"
+		)
+		(instances
+			(project "netdaq"
+				(path "/2970f661-65ab-4e2b-aeda-d76d1044f2b8/944febd4-cf2d-4cdf-a15e-06eb4d902218"
+					(reference "#PWR0552")
+					(unit 1)
+				)
+			)
+		)
+	)
+	(symbol
 		(lib_id "Device:D_TVS")
 		(at 127 199.39 90)
@@
 					(unit 1)
 				)
+			)
+		)
+	)
+	(symbol
+		(lib_id "power:GND")
+		(at 196.85 102.87 0)
+		(mirror x)
+		(unit 1)
+		(body_style 1)
+		(exclude_from_sim no)
+		(in_bom yes)
+		(on_board yes)
+		(in_pos_files yes)
+		(dnp no)
+		(property "Reference" "#PWR0551"
+			(at 196.85 96.52 0)
+			(hide yes)
+			(show_name no)
+			(do_not_autoplace no)
+			(effects
+				(font
+					(size 1.27 1.27)
+				)
+			)
+		)
+		(property "Value" "GND"
+			(at 200.914 101.092 0)
+			(show_name no)
+			(do_not_autoplace no)
+			(effects
+				(font
+					(size 1.27 1.27)
+				)
+			)
+		)
+		(property "Footprint" ""
+			(at 196.85 102.87 0)
+			(hide yes)
+			(show_name no)
+			(do_not_autoplace no)
+			(effects
+				(font
+					(size 1.27 1.27)
+				)
+			)
+		)
+		(property "Datasheet" ""
+			(at 196.85 102.87 0)
+			(hide yes)
+			(show_name no)
+			(do_not_autoplace no)
+			(effects
+				(font
+					(size 1.27 1.27)
+				)
+			)
+		)
+		(property "Description" "Power symbol creates a global label with name \"GND\" , ground"
+			(at 196.85 102.87 0)
+			(hide yes)
+			(show_name no)
+			(do_not_autoplace no)
+			(effects
+				(font
+					(size 1.27 1.27)
+				)
+			)
+		)
+		(pin "1"
+		)
+		(instances
+			(project "netdaq"
+				(path "/2970f661-65ab-4e2b-aeda-d76d1044f2b8/944febd4-cf2d-4cdf-a15e-06eb4d902218"
+					(reference "#PWR0551")
+					(unit 1)
+				)

Commit message: fixed a lot of review comments
Parts:
- D10, D11, D12, D13, D14, D15, D16, D17, D18, D19, D20, D21, D22, D23, D24, D25, D26, D27, D28, D29, D30, D31, D32, D33, D34, D35, D36, D5, D6, D7, D8, D9: value DF2S30FS,L3M -> H24VND3BA; footprint Diode_SMD:D_SOD-923 -> Diode_SMD:D_SOD-323; LCSC C1973663 -> C20615815; LCSC Basic/Pref (none) -> Y; LCSC Part C1973663 -> C20615815

Commit message: pre-changing properties
Parts:
- C100, C39, C40, C43, C44, C47, C48, C51, C52, C55, C56, C59, C60, C63, C64, C67, C68, C71, C72, C75, C76, C79, C80, C83, C84, C87, C88, C91, C92, C95, C96, C99: now left out of the parts list
