File: daq_conn.kicad_sch (KiCad schematic)
At the start: 161 parts, among them J2 DMC 1,5/19-G1F-3,5-LR P26THR

Commit message: did some review cleanup
Parts:
- removed J2: DMC 1,5/19-G1F-3,5-LR P26THR, pxc_1713856_02_01_DMC-1-5-19-G1F-3-5-LR-P26THR:pxc_1713856_02_01_DMC-1-5-19-G1F-3-5-LR-P26THR, symbol pxc_1713856_02_01_DMC-1-5-19-G1F-3-5-LR-P26THR:pxc_1713856_02_01_DMC-1-5-19-G1F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
- added J1: XG4A-5034, CONN_XG4A-5034_OMR, symbol XG4A-5034:XG4A-5034
Connections:
- net ADC1: now also C41.1, R45.1; no longer C38.1, R44.1
- net ADC10: now also C54.1, R52.1; no longer C57.1, R53.1
- net ADC13: now also C65.1, R57.1; no longer C62.1, R56.1
- net ADC14: now also C62.1, R56.1; no longer C65.1, R57.1
- net ADC17: now also C73.1, R61.1; no longer C70.1, R60.1
- net ADC18: now also C70.1, R60.1; no longer C73.1, R61.1
- net ADC2: now also C38.1, R44.1; no longer C41.1, R45.1
- net ADC21: now also C81.1, R65.1; no longer C78.1, R64.1
- net ADC22: now also C78.1, R64.1; no longer C81.1, R65.1
- net ADC25: now also C89.1, R69.1; no longer C86.1, R68.1
- net ADC26: now also C86.1, R68.1; no longer C89.1, R69.1
- net ADC29: now also C97.1, R73.1; no longer C94.1, R72.1
- net ADC30: now also C94.1, R72.1; no longer C97.1, R73.1
- net ADC5: now also C49.1, R49.1; no longer C46.1, R48.1
- net ADC6: now also C46.1, R48.1; no longer C49.1, R49.1
- net ADC9: now also C57.1, R53.1; no longer C54.1, R52.1
- net EXT_ADC1: now also C40.1, D6.2 (A2), R45.2, TP91.1, J1.2; no longer C39.1, D5.2 (A2), R44.2, TP90.1
- net EXT_ADC10: now also C55.1, D13.2 (A2), R52.2, TP98.1, J1.15; no longer C56.1, D14.2 (A2), R53.2, TP99.1
- net EXT_ADC11: now also J1.17
- net EXT_ADC12: now also J1.18
- net EXT_ADC13: now also C64.1, D18.2 (A2), R57.2, TP103.1, J1.20; no longer C63.1, D17.2 (A2), R56.2, TP102.1
- net EXT_ADC14: now also C63.1, D17.2 (A2), R56.2, TP102.1, J1.21; no longer C64.1, D18.2 (A2), R57.2, TP103.1
- net EXT_ADC15: now also J1.23
- net EXT_ADC16: now also J1.24
- net EXT_ADC17: now also C72.1, D22.2 (A2), R61.2, TP107.1, J1.26; no longer C71.1, D21.2 (A2), R60.2, TP106.1
- net EXT_ADC18: now also C71.1, D21.2 (A2), R60.2, TP106.1, J1.27; no longer C72.1, D22.2 (A2), R61.2, TP107.1
- net EXT_ADC19: now also J1.29
- net EXT_ADC2: now also C39.1, D5.2 (A2), R44.2, TP90.1, J1.3; no longer C40.1, D6.2 (A2), R45.2, TP91.1
- net EXT_ADC20: now also J1.30
- net EXT_ADC21: now also C80.1, D26.2 (A2), R65.2, TP111.1, J1.32; no longer C79.1, D25.2 (A2), R64.2, TP110.1
- net EXT_ADC22: now also C79.1, D25.2 (A2), R64.2, TP110.1, J1.33; no longer C80.1, D26.2 (A2), R65.2, TP111.1
- net EXT_ADC23: now also J1.35
- net EXT_ADC24: now also J1.36
- net EXT_ADC25: now also C88.1, D30.2 (A2), R69.2, TP115.1, J1.38; no longer C87.1, D29.2 (A2), R68.2, TP114.1
- net EXT_ADC26: now also C87.1, D29.2 (A2), R68.2, TP114.1, J1.39; no longer C88.1, D30.2 (A2), R69.2, TP115.1
- net EXT_ADC27: now also J1.41
- net EXT_ADC28: now also J1.42
- net EXT_ADC29: now also C96.1, D34.2 (A2), R73.2, TP119.1, J1.44; no longer C95.1, D33.2 (A2), R72.2, TP118.1
- net EXT_ADC3: now also J1.5
- net EXT_ADC30: now also C95.1, D33.2 (A2), R72.2, TP118.1, J1.45; no longer C96.1, D34.2 (A2), R73.2, TP119.1
- net EXT_ADC31: now also J1.47
- net EXT_ADC32: now also J1.48
- net EXT_ADC4: now also J1.6
- net EXT_ADC5: now also C48.1, D10.2 (A2), R49.2, TP95.1, J1.8; no longer C47.1, D9.2 (A2), R48.2, TP94.1
- net EXT_ADC6: now also C47.1, D9.2 (A2), R48.2, TP94.1, J1.9; no longer C48.1, D10.2 (A2), R49.2, TP95.1
- net EXT_ADC7: now also J1.11
- net EXT_ADC8: now also J1.12
- net EXT_ADC9: now also C56.1, D14.2 (A2), R53.2, TP99.1, J1.14; no longer C55.1, D13.2 (A2), R52.2, TP98.1
- net GND: now also J1.1, J1.10, J1.13, J1.16, J1.19, J1.22, J1.25, J1.28, J1.31, J1.34, J1.37, J1.4, J1.40, J1.43, J1.46, J1.49, J1.50, J1.7
Other:
- moved on the sheet: TP100, TP101, TP102, TP103, TP104, TP105, TP106, TP107, TP108, TP109, TP110, TP111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

Commit message: cleaned up the schematic review and cleared ERC
Parts:
- J1: footprint CONN_XG4A-5034_OMR -> XG4A-5034:CONN_XG4A-5034_OMR
Changed lines of the file:
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@@
 		)
 	)
+	(bus
+		(pts
+			(xy 336.55 191.77) (xy 361.95 191.77)
+		)
+		(stroke
+			(width 0)
+			(type default)
+		)
+	)
 	(wire
 		(pts
@@
 		)
 	)
+	(bus
+		(pts
+			(xy 336.55 20.32) (xy 361.95 20.32)
+		)
+		(stroke
+			(width 0)
+			(type default)
+		)
+	)
 	(wire
 		(pts
@@
 		)
 	)
+	(bus
+		(pts
+			(xy 336.55 78.74) (xy 361.95 78.74)
+		)
+		(stroke
+			(width 0)
+			(type default)
+		)
+	)
 	(wire
 		(pts
@@
 		)
 	)
+	(bus
+		(pts
+			(xy 336.55 135.89) (xy 361.95 135.89)
+		)
+		(stroke
+			(width 0)
+			(type default)
+		)
+	)
 	(wire
 		(pts
@@
 		)
 	)
+	(label "ADC[9..16]"
+		(at 361.95 78.74 180)
+		(effects
+			(font
+				(size 1.27 1.27)
+			)
+			(justify right bottom)
+		)
+	)
 	(label "EXT_ADC17"
 		(at 248.92 134.62 180)
@@
 		)
 	)
+	(label "ADC[25..32]"
+		(at 361.95 191.77 180)
+		(effects
+			(font
+				(size 1.27 1.27)
+			)
+			(justify right bottom)
+		)
+	)
 	(label "ADC24"
 		(at 334.01 180.34 180)
@@
 		)
 	)
+	(label "ADC[17..24]"
+		(at 361.95 135.89 180)
+		(effects
+			(font
+				(size 1.27 1.27)
+			)
+			(justify right bottom)
+		)
+	)
 	(label "ADC4"
 		(at 334.01 39.37 180)
@@
 		)
 	)
+	(label "ADC[1..8]"
+		(at 361.95 20.32 180)
+		(effects
+			(font
+				(size 1.27 1.27)
+			)
+			(justify right bottom)
+		)
+	)
 	(label "ADC8"
 		(at 334.01 67.31 180)
@@
 			)
 		)
-		(property "Footprint" "CONN_XG4A-5034_OMR"
+		(property "Footprint" "XG4A-5034:CONN_XG4A-5034_OMR"
 			(at 201.93 104.14 0)
 			(hide yes)
