File: pd_ctrl.kicad_sch (KiCad schematic)
At the start: 13 parts, among them U12 PD70100ILD-TR

Commit message: did some review cleanup
Parts:
- added R278: 33k, Resistor_SMD:R_0402_1005Metric, symbol Device:R
- R260: footprint Resistor_SMD:R_0402_1005Metric -> Resistor_SMD:R_0603_1608Metric
- R91: value 100k -> 150k; footprint Resistor_SMD:R_0402_1005Metric -> Resistor_SMD:R_0603_1608Metric; LCSC C25741 -> C22807; LCSC Part C25741 -> C22807; MPN 0402WGF1003TCE -> 0603WAF1503T5E; Power 62.5mW -> 100mW; Voltage 50V -> 75V
Connections:
- net PD_PG: now also R278.1
- net PGND: now also R278.2
Other:
- note added: "Design Note: 33k/183k: 6.7 V @ 37 V, 10.3 V @ 57 V"
- moved on the sheet: TP215
