File: adc.kicad_sch (KiCad schematic)
At the start: 21 parts, among them U8 TLA2518IRTER

Commit message: did stuff, amongst others changed to op-amp input filter
Parts:
- removed D47, D48, D49, D50, D51, D52, D53, D54: BAS40-04, Package_TO_SOT_SMD:SOT-23, symbol Diode:BAS40-04
- added C131, C150, C167, C168, C205, C206, C207, C208: 10p C0G, Capacitor_SMD:C_0402_1005Metric, symbol Device:C
- added C132, C145, C151, C152, C169, C170, C171, C172, C209, C210, C211, C212, C213, C214, C215, C216: 4.7n C0G, Resistor_SMD:R_0402_1005Metric, symbol Device:C
- added C149, C165, C166, C201, C202, C203, C204, C37: placeholder, symbol Device:C
- added C197, C265: 100n, symbol Device:C
- added D41, D43, D84, D85, D92, D93, D94, D95: BAV199LT1G, C145516:SOT-23_L2.9-W1.3-P1.90-LS2.4-BR, symbol C145516:BAV199LT1G
- added R110, R126, R143, R144, R177, R178, R179, R180: 348k, Resistor_SMD:R_0402_1005Metric, symbol Device:R
- added R111, R121, R127, R128, R145, R146, R147, R148, R181, R182, R183, R184, R185, R186, R187, R188: 1k, Resistor_SMD:R_0402_1005Metric, symbol Device:R
- added R125, R141, R142, R173, R174, R175, R176, R43: 1M, Resistor_SMD:R_0402_1005Metric, symbol Device:R
- added TP183, TP187, TP191, TP192, TP199, TP200, TP201, TP202: TestPoint, TestPoint:TestPoint_THTPad_D1.0mm_Drill0.5mm, symbol Connector:TestPoint
- added U18, U22: TLV9004IPWR, C2058050:TSSOP-14_L5.0-W4.4-P0.65-LS6.4-BL, symbol C2058050:TLV9004IPWR
- U8: footprint TLA2518IRTER:WQFN16_RTE_TEX -> WQFN16_RTE_TEX; LCSC (none) -> C1855741
Connections:
- net GND: now also C131.1, C132.1, C145.1, C150.1, C151.1, C152.1, C167.1, C168.1, C169.1, C170.1, C171.1, C172.1, C197.1, C205.1, C206.1, C207.1, C208.1, C209.1, C210.1, C211.1, C212.1, C213.1, C214.1, C215.1, C216.1, C265.1, D41.1, D43.1, D84.1, D85.1, D92.1, D93.1, D94.1, D95.1, R110.1, R126.1, R143.1, R144.1, R177.1, R178.1, R179.1, R180.1, U18.10 (11), U22.10 (11)
- net GPIO0 renamed INT_ADCIN0
- net INT_ADCIN0: now also C145.2, R121.1
- net GPIO1 renamed INT_ADCIN1
- net INT_ADCIN1: now also C152.2, R128.1
- net GPIO2 renamed INT_ADCIN2
- net INT_ADCIN2: now also C171.2, R147.1
- net GPIO3 renamed INT_ADCIN3
- net INT_ADCIN3: now also C172.2, R148.1
- net GPIO4 renamed INT_ADCIN4
- net INT_ADCIN4: now also C213.2, R185.1
- net GPIO5 renamed INT_ADCIN5
- net INT_ADCIN5: now also C214.2, R186.1
- net GPIO6 renamed INT_ADCIN6
- net INT_ADCIN6: now also C215.2, R187.1
- net GPIO7 renamed INT_ADCIN7
- net INT_ADCIN7: now also C216.2, R188.1
- new net: C169.2, R145.1, R147.2
- new net: C151.2, R127.1, R128.2
- new net: C132.2, R111.1, R121.2
- new net: R182.2, U22.6 (-), U22.7
- new net: R146.2, U18.8, U18.9 (-)
- new net: C209.2, R181.1, R185.2
- new net: R145.2, U18.13 (-), U18.14
- new net: C211.2, R183.1, R187.2
- new net: C210.2, R182.1, R186.2
- new net: R181.2, U22.1, U22.2 (-)
- new net: C170.2, R146.1, R148.2
- new net: R184.2, U22.8, U22.9 (-)
- new net: R183.2, U22.13 (-), U22.14
- new net: R127.2, U18.6 (-), U18.7
- new net: C212.2, R184.1, R188.2
- new net: R111.2, U18.1, U18.2 (-)
- new net +3.3V: C197.2, C265.2, D41.2, D43.2, D84.2, D85.2, D92.2, D93.2, D94.2, D95.2, U18.4 (V+), U22.4 (V+)
- new net ADCIN0: C37.2, R43.2
- new net ADCIN1: C149.2, R125.2
- new net ADCIN2: C165.2, R141.2
- new net ADCIN3: C166.2, R142.2
- new net ADCIN4: C201.2, R173.2
- new net ADCIN5: C202.2, R174.2
- new net ADCIN6: C203.2, R175.2
- new net ADCIN7: C204.2, R176.2
- new net ADCIN_SCALED0: C131.2, C37.1, D41.3, R110.2, R43.1, TP183.1, U18.3 (+)
- new net ADCIN_SCALED1: C149.1, C150.2, D43.3, R125.1, R126.2, TP187.1, U18.5 (+)
- new net ADCIN_SCALED2: C165.1, C167.2, D84.3, R141.1, R143.2, TP191.1, U18.12 (+)
- new net ADCIN_SCALED3: C166.1, C168.2, D85.3, R142.1, R144.2, TP192.1, U18.10 (+)
- new net ADCIN_SCALED4: C201.1, C205.2, D92.3, R173.1, R177.2, TP199.1, U22.3 (+)
- new net ADCIN_SCALED5: C202.1, C206.2, D93.3, R174.1, R178.2, TP200.1, U22.5 (+)
- new net ADCIN_SCALED6: C203.1, C207.2, D94.3, R175.1, R179.2, TP201.1, U22.12 (+)
- new net ADCIN_SCALED7: C204.1, C208.2, D95.3, R176.1, R180.2, TP202.1, U22.10 (+)
Other:
- moved on the sheet: C115, C116, C117, TP136, TP137, TP138, TP139, TP140, TP141, TP142, TP143, TP144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

Commit message: fixed couple of things
Connections:
- net +3.3V: now also C116.1, C117.1, U8.10 (DVDD), U8.7 (AVDD)
- net GND: now also U18.11 (V-), U22.11 (V-); no longer U18.10 (11), U22.10 (11)
Changed lines of the file:
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@@
 	)
 	(junction
+		(at 363.22 158.75)
+		(diameter 0)
+		(color 0 0 0 0)
+	)
+	(junction
 		(at 107.95 87.63)
 		(diameter 0)
@@
 	)
 	(junction
+		(at 373.38 154.94)
+		(diameter 0)
+		(color 0 0 0 0)
+	)
+	(junction
 		(at 121.92 194.31)
 		(diameter 0)
@@
 	)
 	(junction
+		(at 373.38 158.75)
+		(diameter 0)
+		(color 0 0 0 0)
+	)
+	(junction
 		(at 107.95 114.3)
 		(diameter 0)
@@
 	(wire
 		(pts
+			(xy 373.38 158.75) (xy 373.38 168.91)
+		)
+		(stroke
+			(width 0)
+			(type default)
+		)
+	)
+	(wire
+		(pts
 			(xy 190.5 34.29) (xy 246.38 34.29)
 		)
@@
 	(wire
 		(pts
+			(xy 363.22 158.75) (xy 373.38 158.75)
+		)
+		(stroke
+			(width 0)
+			(type default)
+		)
+	)
+	(wire
+		(pts
 			(xy 113.03 231.14) (xy 113.03 232.41)
 		)
@@
 	(wire
 		(pts
+			(xy 373.38 152.4) (xy 373.38 154.94)
+		)
+		(stroke
+			(width 0)
+			(type default)
+		)
+	)
+	(wire
+		(pts
 			(xy 97.79 95.25) (xy 95.25 95.25)
 		)
@@
 	(wire
 		(pts
-			(xy 373.38 154.94) (xy 373.38 168.91)
+			(xy 373.38 154.94) (xy 373.38 158.75)
 		)
 		(stroke
@@
 		(pin "10"
 		)
-		(pin "10"
+		(pin "11"
 		)
 		(instances
@@
 		(pin "10"
 		)
-		(pin "10"
+		(pin "11"
 		)
 		(instances
@@
 	)
 	(symbol
+		(lib_id "power:+3.3V")
+		(at 373.38 152.4 0)
+		(mirror y)
+		(unit 1)
+		(body_style 1)
+		(exclude_from_sim no)
+		(in_bom yes)
+		(on_board yes)
+		(in_pos_files yes)
+		(dnp no)
+		(property "Reference" "#PWR0200"
+			(at 373.38 156.21 0)
+			(hide yes)
+			(show_name no)
+			(do_not_autoplace no)
+			(effects
+				(font
+					(size 1.27 1.27)
+				)
+			)
+		)
+		(property "Value" "+3.3V"
+			(at 377.444 150.622 0)
+			(show_name no)
+			(do_not_autoplace no)
+			(effects
+				(font
+					(size 1.27 1.27)
+				)
+			)
+		)
+		(property "Footprint" ""
+			(at 373.38 152.4 0)
+			(hide yes)
+			(show_name no)
+			(do_not_autoplace no)
+			(effects
+				(font
+					(size 1.27 1.27)
+				)
+			)
+		)
+		(property "Datasheet" ""
+			(at 373.38 152.4 0)
+			(hide yes)
+			(show_name no)
+			(do_not_autoplace no)
+			(effects
+				(font
+					(size 1.27 1.27)
+				)
+			)
+		)
+		(property "Description" "Power symbol creates a global label with name \"+3.3V\""
+			(at 373.38 152.4 0)
+			(hide yes)
+			(show_name no)
+			(do_not_autoplace no)
+			(effects
+				(font
+					(size 1.27 1.27)
+				)
+			)
+		)
+		(pin "1"
+		)
+		(instances
+			(project "netdaq"
+				(path "/2970f661-65ab-4e2b-aeda-d76d1044f2b8/1b815250-feab-4e15-9fc8-1220df09f4d5"
+					(reference "#PWR0201")
+					(unit 1)
+				)
+				(path "/2970f661-65ab-4e2b-aeda-d76d1044f2b8/443c8de8-4114-4248-9fe3-e4e39d7e1ee6"
+					(reference "#PWR0202")
+					(unit 1)
+				)
+				(path "/2970f661-65ab-4e2b-aeda-d76d1044f2b8/8ecbce95-7163-4b25-8ea0-7aacaf2b4420"
+					(reference "#PWR0200")
+					(unit 1)
+				)
+				(path "/2970f661-65ab-4e2b-aeda-d76d1044f2b8/b1f1b5cf-56ac-4b0f-bbb9-08aecf979a8c"
+					(reference "#PWR0203")
+					(unit 1)
+				)
+			)
+		)
+	)
+	(symbol
 		(lib_id "C145516:BAV199LT1G")
 		(at 130.81 34.29 270)
@@
 		(pin "10"
 		)
-		(pin "10"
+		(pin "11"
 		)
 		(instances
@@
 		(pin "10"
 		)
-		(pin "10"
+		(pin "11"
 		)
 		(instances
@@
 		(pin "10"
 		)
-		(pin "10"
+		(pin "11"
 		)
 		(instances
@@
 		(pin "10"
 		)
-		(pin "10"
+		(pin "11"
 		)
 		(instances
@@
 		(pin "10"
 		)
-		(pin "10"
+		(pin "11"
 		)
 		(instances
@@
 		(pin "10"
 		)
-		(pin "10"
+		(pin "11"
 		)
 		(instances
@@
 		(pin "10"
 		)
-		(pin "10"
+		(pin "11"
 		)
 		(instances
@@
 		(pin "10"
 		)
-		(pin "10"
+		(pin "11"
 		)
 		(instances
