File: adc.kicad_sch (KiCad schematic)
At the start: 97 parts, among them U18 TLV9004IPWR, U22 TLV9004IPWR, U8 TLA2518IRTER

Commit message: fixed some more schematic review
Parts:
- added C281: 100n 50V, Capacitor_SMD:C_0402_1005Metric, symbol Device:C
- added R272: 10k, Resistor_SMD:R_0402_1005Metric, symbol Device:R
- R110, R126, R143, R144, R177, R178, R179, R180: value 348k -> 309k; LCSC C4135252 -> C4180598; LCSC Part C4135252 -> C4180598; MPN RE0402BRE07348KL -> RE0402BRE07309KL
Connections:
- net +3.3V: now also R272.1; no longer C117.1, U8.7 (AVDD)
- net GND: now also C281.2
- net SPI.CS#: now also R272.2
- new net +3.0V_REF: C117.1, C281.1, U8.7 (AVDD)

Commit message: did some review cleanup
Parts:
- U8: footprint WQFN16_RTE_TEX -> TLA2518IRTER:WQFN16_RTE_TEX
Changed lines of the file:
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@@
 			)
 		)
-		(property "Footprint" "WQFN16_RTE_TEX"
+		(property "Footprint" "TLA2518IRTER:WQFN16_RTE_TEX"
 			(at 276.86 118.11 0)
 			(hide yes)
