File: debug_conn.kicad_sch (KiCad schematic)
At the start: 22 parts, among them CN1 HX JN1.27-2x5P ZZ H4.9, J3 2.54-1x6PStraight pin, U14 TXU0202DCUR, U26 TLV77033PDBVR

Commit message: fixed some more schematic review
Connections:
- net +3.3V: no longer R96.1
- net GND: now also R96.2
- net JTAG.TCK: now also R96.1; no longer R96.2

Commit message: cleaned up the schematic review and cleared ERC
Changed lines of the file:
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@@
 	)
 	(junction
+		(at 171.45 57.15)
+		(diameter 0)
+		(color 0 0 0 0)
+	)
+	(junction
 		(at 158.75 137.16)
 		(diameter 0)
@@
 	(wire
 		(pts
-			(xy 171.45 59.69) (xy 171.45 48.26)
+			(xy 171.45 59.69) (xy 171.45 57.15)
 		)
 		(stroke
@@
 	(wire
 		(pts
+			(xy 171.45 57.15) (xy 171.45 48.26)
+		)
+		(stroke
+			(width 0)
+			(type default)
+		)
+	)
+	(wire
+		(pts
 			(xy 151.13 132.08) (xy 151.13 139.7)
 		)
@@
 					(unit 1)
 				)
+			)
+		)
+	)
+	(symbol
+		(lib_id "power:PWR_FLAG")
+		(at 171.45 57.15 90)
+		(unit 1)
+		(body_style 1)
+		(exclude_from_sim no)
+		(in_bom yes)
+		(on_board yes)
+		(in_pos_files yes)
+		(dnp no)
+		(fields_autoplaced yes)
+		(property "Reference" "#FLG07"
+			(at 169.545 57.15 0)
+			(hide yes)
+			(show_name no)
+			(do_not_autoplace no)
+			(effects
+				(font
+					(size 1.27 1.27)
+				)
+			)
+		)
+		(property "Value" "PWR_FLAG"
+			(at 167.64 57.1499 90)
+			(show_name no)
+			(do_not_autoplace no)
+			(effects
+				(font
+					(size 1.27 1.27)
+				)
+				(justify left)
+			)
+		)
+		(property "Footprint" ""
+			(at 171.45 57.15 0)
+			(hide yes)
+			(show_name no)
+			(do_not_autoplace no)
+			(effects
+				(font
+					(size 1.27 1.27)
+				)
+			)
+		)
+		(property "Datasheet" ""
+			(at 171.45 57.15 0)
+			(hide yes)
+			(show_name no)
+			(do_not_autoplace no)
+			(effects
+				(font
+					(size 1.27 1.27)
+				)
+			)
+		)
+		(property "Description" "Special symbol for telling ERC where power comes from"
+			(at 171.45 57.15 0)
+			(hide yes)
+			(show_name no)
+			(do_not_autoplace no)
+			(effects
+				(font
+					(size 1.27 1.27)
+				)
+			)
+		)
+		(pin "1"
+		)
+		(instances
+			(project "netdaq"
+				(path "/2970f661-65ab-4e2b-aeda-d76d1044f2b8/3126208c-7808-4087-8557-46cefae30ae4"
+					(reference "#FLG07")
+					(unit 1)
+				)
