File: sdmmc.kicad_sch (KiCad schematic)
At the start: 12 parts, among them U15 MLD-TF PUSH-H18, U16 TPUSBLC6-4SC6, U17 TPUSBLC6-4SC6

Commit message: fixed some more schematic review
Parts:
- R87: now not fitted
- U16, U17: symbol Library:TPUSBLC6-4SC6 -> TPUSBLC6:TPUSBLC6-4SC6
Changed lines of the file:
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@@
 	)
 	(symbol
-		(lib_id "Library:TPUSBLC6-4SC6")
+		(lib_id "TPUSBLC6:TPUSBLC6-4SC6")
 		(at 170.18 124.46 0)
 		(unit 1)
@@
 		(on_board yes)
 		(in_pos_files yes)
-		(dnp no)
+		(dnp yes)
 		(fields_autoplaced yes)
 		(property "Reference" "R87"
@@
 	)
 	(symbol
-		(lib_id "Library:TPUSBLC6-4SC6")
+		(lib_id "TPUSBLC6:TPUSBLC6-4SC6")
 		(at 130.81 124.46 0)
 		(unit 1)

Commit message: did some review cleanup
Parts:
- R87: now left out of the parts list
Changed lines of the file:
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@@
 		(body_style 1)
 		(exclude_from_sim no)
-		(in_bom yes)
+		(in_bom no)
 		(on_board yes)
 		(in_pos_files yes)
