File: eeprom.kicad_sch (KiCad schematic)
At the start: 10 parts, among them U29 M24C64-RMN6TP

Commit message: cleaned up the schematic review and cleared ERC
Parts:
- removed R2, R280, R282: 10k, Resistor_SMD:R_0402_1005Metric, symbol Device:R
- R284: now not fitted; now left out of the parts list
Other:
- note added: "DNM"
