File: usb_conn.kicad_sch (KiCad schematic)
At the start: 16 parts, among them U13 DLM0NSN500HY2D, U6 TPUSBLC6-4SC6

Commit message: fixed some more schematic review
Parts:
- added R276: 10k, Resistor_SMD:R_0402_1005Metric, symbol Device:R
- U6: symbol Library:TPUSBLC6-4SC6 -> TPUSBLC6:TPUSBLC6-4SC6
Connections:
- net GND: now also R276.2; no longer USB1.1 (SHELL), USB1.2 (SHELL), USB1.3 (SHELL), USB1.4 (SHELL)
- new net USB_SHIELD: R276.1, USB1.1 (SHELL), USB1.2 (SHELL), USB1.3 (SHELL), USB1.4 (SHELL)

Commit message: cleaned up the schematic review and cleared ERC
Changed lines of the file:
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@@
 	)
 	(junction
+		(at 101.6 86.36)
+		(diameter 0)
+		(color 0 0 0 0)
+	)
+	(junction
 		(at 189.23 86.36)
 		(diameter 0)
@@
 	(wire
 		(pts
+			(xy 101.6 86.36) (xy 107.95 86.36)
+		)
+		(stroke
+			(width 0)
+			(type default)
+		)
+	)
+	(wire
+		(pts
 			(xy 217.17 106.68) (xy 214.63 106.68)
 		)
@@
 	(wire
 		(pts
-			(xy 92.71 86.36) (xy 107.95 86.36)
+			(xy 92.71 86.36) (xy 101.6 86.36)
 		)
 		(stroke
@@
 	)
 	(symbol
+		(lib_id "power:PWR_FLAG")
+		(at 101.6 86.36 0)
+		(unit 1)
+		(body_style 1)
+		(exclude_from_sim no)
+		(in_bom yes)
+		(on_board yes)
+		(in_pos_files yes)
+		(dnp no)
+		(fields_autoplaced yes)
+		(property "Reference" "#FLG08"
+			(at 101.6 84.455 0)
+			(hide yes)
+			(show_name no)
+			(do_not_autoplace no)
+			(effects
+				(font
+					(size 1.27 1.27)
+				)
+			)
+		)
+		(property "Value" "PWR_FLAG"
+			(at 101.6 81.28 0)
+			(show_name no)
+			(do_not_autoplace no)
+			(effects
+				(font
+					(size 1.27 1.27)
+				)
+			)
+		)
+		(property "Footprint" ""
+			(at 101.6 86.36 0)
+			(hide yes)
+			(show_name no)
+			(do_not_autoplace no)
+			(effects
+				(font
+					(size 1.27 1.27)
+				)
+			)
+		)
+		(property "Datasheet" ""
+			(at 101.6 86.36 0)
+			(hide yes)
+			(show_name no)
+			(do_not_autoplace no)
+			(effects
+				(font
+					(size 1.27 1.27)
+				)
+			)
+		)
+		(property "Description" "Special symbol for telling ERC where power comes from"
+			(at 101.6 86.36 0)
+			(hide yes)
+			(show_name no)
+			(do_not_autoplace no)
+			(effects
+				(font
+					(size 1.27 1.27)
+				)
+			)
+		)
+		(pin "1"
+		)
+		(instances
+			(project "netdaq"
+				(path "/2970f661-65ab-4e2b-aeda-d76d1044f2b8/c9141396-b417-45d3-9560-a5d378bd1b7a"
+					(reference "#FLG08")
+					(unit 1)
+				)
+			)
+		)
+	)
+	(symbol
 		(lib_id "power:+1V0")
 		(at 92.71 83.82 0)
@@
 		)
 		(property "Footprint" "Resistor_SMD:R_0402_1005Metric"
-			(at 121.92 88.138 90)
+			(at 124.206 98.552 90)
 			(hide yes)
 			(show_name no)
@@
 		)
 		(property "Datasheet" "https://datasheet.lcsc.com/datasheet/pdf/f85b01b3a1a015a5ec4a9f03876e0063.pdf?productCode=C85813"
-			(at 121.92 86.36 0)
+			(at 102.362 85.598 0)
 			(hide yes)
 			(show_name no)
@@
 		)
 		(property "Description" "Ferrite bead"
-			(at 121.92 86.36 0)
+			(at 115.824 102.87 0)
 			(hide yes)
 			(show_name no)
@@
 		)
 		(property "LCSC Part" "C85813"
-			(at 121.92 86.36 90)
+			(at 122.428 99.314 90)
 			(hide yes)
 			(show_name no)
@@
 		)
 		(property "MPN" "BLM15AG221SN1D"
-			(at 121.92 86.36 90)
+			(at 123.19 101.854 90)
 			(hide yes)
 			(show_name no)
